File: Eagle/MSGP/MSGP.brd (EAGLE design)
At the start: 100 x 80 mm, 13 parts, among them T1 2N3904

Commit message: MSBP board
Parts:
- removed C6: (no value), rcl:C050-045X075
- added C7, C8: (no value), rcl:C050-045X075
- added R5: (no value), rcl:0207/10
- moved C2 79.1 mm to (64.8, 76.2), turned to 0 degrees
- moved C1 76.1 mm to (73.7, 55.9), turned to 90 degrees
- moved C3 67.7 mm to (64.8, 63.5), turned to 0 degrees
- moved T1 52.5 mm to (62.2, 44.5), turned to 270 degrees
- moved L1 50.3 mm to (55.9, 68.6), turned to 90 degrees
- moved U$1 38.6 mm to (62.2, 25.4)
- moved C4 38.6 mm to (55.9, 55.9), turned to 90 degrees
- moved C5 37.8 mm to (69.8, 35.6), turned to 180 degrees
- moved R3 29.0 mm to (38.1, 61.0), turned to 180 degrees
- moved R2 16.6 mm to (44.5, 49.5)
- moved R4 11.4 mm to (25.4, 29.2), turned to 180 degrees
- moved R1 4.02 mm to (33.0, 49.5)
Connections:
- removed net N$7: C6.1, U$1.5
- new net N$6: C5.1, U$1.2, U$1.6
- new net N$9: C8.1, R5.2
- net GND: now also C7.2, C8.2; no longer C6.2
- net N$1: now also R5.1; no longer C5.1, U$1.6
- net VCC: now also C7.1, U$1.4
Routing:
- net VCC: track 0.00 -> 100.7 mm
- net N$1: track 0.00 -> 66.7 mm
- net N$5: track 0.00 -> 46.6 mm
- net N$3: track 0.00 -> 46.0 mm
- net N$6: track 0.00 -> 28.4 mm
- net N$9: track 0.00 -> 23.7 mm
- net GND: track 0.00 -> 12.0 mm
- net N$4: track 0.00 -> 11.4 mm
- net N$2: track 0.00 -> 6.84 mm
- added copper zone on layer 1, net GND
Other:
- board size 100 x 80 mm -> 100 x 83.8 mm

Commit message: new MSGP
Parts:
- removed C1, C2, C3, C4, C5, C7, C8: (no value), rcl:C050-045X075
- removed L1, R1, R2, R3, R4, R5: (no value), rcl:0207/10
- removed T1: 2N3904, transistor-neu-to92:TO92
- removed U$1: LMC555, E3VB_ISI:8-DIP
- added IC1: 74ALS04D, 74xx-us:SO14
- added U1: LTC6905CS5TRMPBF, LTC_By_element14_Batch_1:SOT95P280X100-5N
Connections:
- removed net N$1: R4.1, R5.1, U$1.7
- removed net N$2: C2.1, L1.2
- removed net N$3: C4.1, R1.2, R2.2, R3.1, T1.1
- removed net N$4: C3.1, C4.2, L1.1
- removed net N$5: C1.1, R1.1, R2.1, T1.2
- removed net N$6: C5.1, U$1.2, U$1.6
- removed net N$9: C8.1, R5.2
- new net V+: U1.1
- net GND: now also IC1.7; no longer C1.2, C2.2, C3.2, C5.2, C7.2, C8.2, T1.3, U$1.1
- net VCC: now also IC1.14; no longer C7.1, R3.2, R4.2, U$1.4, U$1.8
Routing:
- net VCC: track 100.7 -> 0.00 mm
- net N$1: track 66.7 -> 0.00 mm
- net N$5: track 46.6 -> 0.00 mm
- net N$3: track 46.0 -> 0.00 mm
- net N$6: track 28.4 -> 0.00 mm
- net N$9: track 23.7 -> 0.00 mm
- net GND: track 12.0 -> 0.00 mm
- net N$4: track 11.4 -> 0.00 mm
- net N$2: track 6.84 -> 0.00 mm
Changed lines of the file:
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@@
 </autorouter>
 <elements>
-<element name="C1" library="rcl" package="C050-045X075" value="" x="73.66" y="55.88" rot="R90"/>
-<element name="C2" library="rcl" package="C050-045X075" value="" x="64.77" y="76.2"/>
-<element name="C3" library="rcl" package="C050-045X075" value="" x="64.77" y="63.5"/>
-<element name="C4" library="rcl" package="C050-045X075" value="" x="55.88" y="55.88" rot="R90"/>
-<element name="C5" library="rcl" package="C050-045X075" value="" x="69.85" y="35.56" rot="R180"/>
-<element name="L1" library="rcl" package="0207/10" value="" x="55.88" y="68.58" rot="R90"/>
-<element name="R1" library="rcl" package="0207/10" value="" x="33.02" y="49.53" rot="R90"/>
-<element name="R2" library="rcl" package="0207/10" value="" x="44.45" y="49.53" rot="R90"/>
-<element name="R3" library="rcl" package="0207/10" value="" x="38.1" y="60.96" rot="R180"/>
-<element name="R4" library="rcl" package="0207/10" value="" x="25.4" y="29.21" rot="R180"/>
-<element name="T1" library="transistor-neu-to92" package="TO92" value="2N3904" x="62.23" y="44.45" rot="R270"/>
-<element name="U$1" library="E3VB_ISI" package="8-DIP" value="LMC555" x="62.23" y="25.4" rot="R270"/>
-<element name="R5" library="rcl" package="0207/10" value="" x="66.04" y="10.16" rot="R180"/>
-<element name="C7" library="rcl" package="C050-045X075" value="" x="20.32" y="44.45" rot="R90"/>
-<element name="C8" library="rcl" package="C050-045X075" value="" x="38.1" y="19.05" rot="R90"/>
+<element name="IC1" library="74xx-us" package="SO14" value="74ALS04D" x="6.604" y="-5.08"/>
+<element name="U1" library="LTC_By_element14_Batch_1" package="SOT95P280X100-5N" value="LTC6905CS5TRMPBF" x="4.318" y="-14.732">
+<attribute name="PACKAGE" value="SOT-23-5" x="4.318" y="-14.732" size="1.778" layer="27" display="off"/>
+<attribute name="OC_NEWARK" value="19P0750" x="4.318" y="-14.732" size="1.778" layer="27" display="off"/>
+<attribute name="MPN" value="LTC6905CS5#TRMPBF" x="4.318" y="-14.732" size="1.778" layer="27" display="off"/>
+<attribute name="SUPPLIER" value="Linear Technology" x="4.318" y="-14.732" size="1.778" layer="27" display="off"/>
+<attribute name="OC_FARNELL" value="1663923" x="4.318" y="-14.732" size="1.778" layer="27" display="off"/>
+</element>
 </elements>
 <signals>
+<signal name="GND">
+<polygon width="0.4064" layer="1">
+<vertex x="1.016" y="82.804"/>
+<vertex x="98.044" y="82.804"/>
+<vertex x="98.044" y="40.64"/>
+<vertex x="32.512" y="40.64"/>
+<vertex x="32.512" y="15.24"/>
+<vertex x="1.016" y="15.24"/>
+</polygon>
+<polygon width="0.4064" layer="1">
+<vertex x="1.27" y="14.478"/>
+<vertex x="33.782" y="14.478"/>
+<vertex x="33.528" y="39.878"/>
+<vertex x="98.298" y="39.878"/>
+<vertex x="98.298" y="0.508"/>
+<vertex x="1.016" y="0.762"/>
+<vertex x="1.016" y="14.478"/>
+</polygon>
+<contactref element="IC1" pad="7"/>
+</signal>
 <signal name="VCC">
-<contactref element="R3" pad="2"/>
-<contactref element="U$1" pad="8"/>
-<contactref element="R4" pad="2"/>
-<contactref element="C7" pad="1"/>
-<contactref element="U$1" pad="4"/>
-<wire x1="20.32" y1="29.21" x2="20.32" y2="41.91" width="0.4064" layer="1"/>
-<wire x1="20.32" y1="29.21" x2="22.86" y2="25.4" width="0.4064" layer="1"/>
-<wire x1="22.86" y1="25.4" x2="48.26" y2="25.4" width="0.4064" layer="1"/>
-<wire x1="48.26" y1="25.4" x2="52.07" y2="20.32" width="0.4064" layer="1"/>
-<wire x1="52.07" y1="20.32" x2="58.42" y2="20.32" width="0.4064" layer="1"/>
-<wire x1="66.04" y1="27.94" x2="66.04" y2="30.48" width="0.4064" layer="1"/>
-<wire x1="66.04" y1="30.48" x2="53.34" y2="30.48" width="0.4064" layer="1"/>
-<wire x1="53.34" y1="30.48" x2="48.26" y2="25.4" width="0.4064" layer="1"/>
-<wire x1="20.32" y1="41.91" x2="33.02" y2="60.96" width="0.4064" layer="16"/>
+<contactref element="IC1" pad="14"/>
 </signal>
-<signal name="N$2">
-<contactref element="C2" pad="1"/>
-<contactref element="L1" pad="2"/>
-<wire x1="55.88" y1="73.66" x2="62.23" y2="76.2" width="0.4064" layer="16"/>
-</signal>
-<signal name="N$3">
-<contactref element="R3" pad="1"/>
-<contactref element="T1" pad="1"/>
-<contactref element="R2" pad="2"/>
-<contactref element="R1" pad="2"/>
-<contactref element="C4" pad="1"/>
-<wire x1="33.02" y1="54.61" x2="44.45" y2="54.61" width="0.4064" layer="1"/>
-<wire x1="43.18" y1="60.96" x2="44.45" y2="60.96" width="0.4064" layer="1"/>
-<wire x1="44.45" y1="60.96" x2="44.45" y2="54.61" width="0.4064" layer="1"/>
-<wire x1="44.45" y1="54.61" x2="54.61" y2="54.61" width="0.4064" layer="1"/>
-<wire x1="54.61" y1="54.61" x2="55.88" y2="53.34" width="0.4064" layer="1"/>
-<wire x1="62.23" y1="43.18" x2="58.42" y2="43.18" width="0.4064" layer="1"/>
-<wire x1="58.42" y1="43.18" x2="55.88" y2="45.72" width="0.4064" layer="1"/>
-<wire x1="55.88" y1="45.72" x2="55.88" y2="53.34" width="0.4064" layer="1"/>
-</signal>
-<signal name="GND">
-<contactref element="U$1" pad="1"/>
-<contactref element="C1" pad="2"/>
-<contactref element="C5" pad="2"/>
-<contactref element="T1" pad="3"/>
-<contactref element="C2" pad="2"/>
-<contactref element="C3" pad="2"/>
-<contactref element="C7" pad="2"/>
-<contactref element="C8" pad="2"/>
-<polygon width="0.4064" layer="1" isolate="1.27">
-<vertex x="2.54" y="81.28"/>
-<vertex x="97.79" y="81.28"/>
-<vertex x="97.79" y="2.54"/>
-<vertex x="2.54" y="2.54"/>
-</polygon>
-<wire x1="67.31" y1="35.56" x2="66.04" y2="35.56" width="0.4064" layer="16"/>
-<wire x1="66.04" y1="35.56" x2="58.42" y2="27.94" width="0.4064" layer="16"/>
-</signal>
-<signal name="N$5">
-<contactref element="T1" pad="2"/>
-<contactref element="R1" pad="1"/>
-<contactref element="R2" pad="1"/>
-<contactref element="C1" pad="1"/>
-<wire x1="33.02" y1="44.45" x2="44.45" y2="44.45" width="0.4064" layer="1"/>
-<wire x1="73.66" y1="53.34" x2="73.66" y2="49.53" width="0.4064" layer="1"/>
-<wire x1="73.66" y1="49.53" x2="68.58" y2="44.45" width="0.4064" layer="1"/>
-<wire x1="68.58" y1="44.45" x2="64.262" y2="44.45" width="0.4064" layer="1"/>
-<wire x1="64.262" y1="44.45" x2="44.45" y2="44.45" width="0.4064" layer="16"/>
-<wire x1="64.262" y1="44.45" x2="64.135" y2="44.45" width="0" layer="19" extent="1-1"/>
-<wire x1="64.262" y1="44.45" x2="64.262" y2="44.45" width="0" layer="19" extent="1-16"/>
-</signal>
-<signal name="N$4">
-<contactref element="C3" pad="1"/>
-<contactref element="L1" pad="1"/>
-<contactref element="C4" pad="2"/>
-<wire x1="55.88" y1="63.5" x2="62.23" y2="63.5" width="0.4064" layer="16"/>
-<wire x1="55.88" y1="58.42" x2="55.88" y2="63.5" width="0.4064" layer="16"/>
-</signal>
-<signal name="N$1">
-<contactref element="U$1" pad="7"/>
-<contactref element="R5" pad="1"/>
-<contactref element="R4" pad="1"/>
-<wire x1="66.04" y1="25.4" x2="68.58" y2="25.4" width="0.4064" layer="1"/>
-<wire x1="68.58" y1="25.4" x2="71.12" y2="27.94" width="0.4064" layer="1"/>
-<wire x1="71.12" y1="27.94" x2="67.31" y2="31.75" width="0.4064" layer="1"/>
-<wire x1="67.31" y1="31.75" x2="33.02" y2="31.75" width="0.4064" layer="1"/>
-<wire x1="33.02" y1="31.75" x2="30.48" y2="29.21" width="0.4064" layer="1"/>
-<wire x1="71.12" y1="10.16" x2="71.12" y2="20.32" width="0.4064" layer="16"/>
-<wire x1="71.12" y1="20.32" x2="66.04" y2="25.4" width="0.4064" layer="16"/>
-</signal>
-<signal name="N$6">
-<contactref element="C5" pad="1"/>
-<contactref element="U$1" pad="6"/>
-<contactref element="U$1" pad="2"/>
-<wire x1="58.42" y1="25.4" x2="66.04" y2="22.86" width="0.4064" layer="1"/>
-<wire x1="72.39" y1="35.56" x2="74.93" y2="33.02" width="0.4064" layer="1"/>
-<wire x1="74.93" y1="33.02" x2="74.93" y2="26.67" width="0.4064" layer="1"/>
-<wire x1="74.93" y1="26.67" x2="71.12" y2="22.86" width="0.4064" layer="1"/>
-<wire x1="71.12" y1="22.86" x2="66.04" y2="22.86" width="0.4064" layer="1"/>
-</signal>
-<signal name="N$9">
-<contactref element="R5" pad="2"/>
-<contactref element="C8" pad="1"/>
-<wire x1="38.1" y1="16.51" x2="60.96" y2="10.16" width="0.4064" layer="1"/>
+<signal name="V+">
+<contactref element="U1" pad="1"/>
 </signal>
 </signals>
