File: Eagle/MSGP/MSGP.brd (EAGLE design)
At the start: 71.8 x 43.9 mm, 27 parts, among them IC1 74ALS04D, IC2 NE5532D, U1 LTC6905CS5TRMPBF

Commit message: Updated Schematic
Parts:
- removed JP3: (no value), jumper:JP1
- moved JP7 96.1 mm to (54.6, 31.8), turned to 270 degrees
- moved R11 74.3 mm to (44.5, 30.5), turned to 90 degrees
- moved R10 70.1 mm to (39.4, 35.6), turned to 90 degrees
Connections:
- removed net N$14: JP3.2, R10.1, R11.2
- net GND: no longer JP3.1
- net N$2: now also R10.1, R11.2
Routing:
- net N$12: track 0.00 -> 36.0 mm
- net N$2: track 13.1 -> 32.6 mm
- net N$13: track 0.00 -> 13.6 mm
Changed lines of the file:
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@@
 <element name="R8" library="resistor" package="0204V" value="" x="11.43" y="34.798" rot="R180"/>
 <element name="R9" library="resistor" package="0204V" value="" x="7.874" y="31.496" rot="R270"/>
-<element name="R10" library="resistor" package="0204V" value="" x="-17.78" y="-5.08"/>
-<element name="R11" library="resistor" package="0204V" value="" x="-17.78" y="-10.16"/>
-<element name="JP3" library="jumper" package="JP1" value="" x="-25.4" y="-7.62"/>
-<element name="JP7" library="jumper" package="JP1" value="" x="-33.02" y="-7.62"/>
+<element name="R10" library="resistor" package="0204V" value="" x="39.37" y="35.56" rot="R90"/>
+<element name="R11" library="resistor" package="0204V" value="" x="44.45" y="30.48" rot="R90"/>
+<element name="JP7" library="jumper" package="JP1" value="" x="54.61" y="31.75" rot="R270"/>
 </elements>
 <signals>
@@
 </polygon>
 <contactref element="IC2" pad="5"/>
-<contactref element="JP3" pad="1"/>
 <contactref element="JP7" pad="2"/>
-<wire x1="62.992" y1="8.128" x2="62.23" y2="18.034" width="0" layer="19" extent="1-1"/>
-<wire x1="44.764" y1="23.241" x2="62.23" y2="18.034" width="0" layer="19" extent="1-1"/>
-<wire x1="44.764" y1="24.511" x2="44.764" y2="23.241" width="0" layer="19" extent="1-1"/>
-<wire x1="39.564" y1="24.511" x2="44.764" y2="24.511" width="0" layer="19" extent="1-1"/>
-<wire x1="34.29" y1="29.718" x2="39.564" y2="24.511" width="0" layer="19" extent="1-1"/>
-<wire x1="31.75" y1="29.718" x2="34.29" y2="29.718" width="0" layer="19" extent="1-1"/>
-<wire x1="29.464" y1="32.766" x2="31.75" y2="29.718" width="0" layer="19" extent="1-1"/>
-<wire x1="29.718" y1="35.814" x2="29.464" y2="32.766" width="0" layer="19" extent="1-1"/>
-<wire x1="29.21" y1="39.624" x2="29.718" y2="35.814" width="0" layer="19" extent="1-1"/>
-<wire x1="22.8854" y1="37.846" x2="29.21" y2="39.624" width="0" layer="19" extent="1-1"/>
-<wire x1="41.91" y1="13.97" x2="44.764" y2="23.241" width="0" layer="19" extent="1-1"/>
-<wire x1="35.814" y1="6.374" x2="41.91" y2="13.97" width="0" layer="19" extent="1-1"/>
-<wire x1="30.988" y1="6.374" x2="35.814" y2="6.374" width="0" layer="19" extent="1-1"/>
-<wire x1="21.59" y1="6.628" x2="30.988" y2="6.374" width="0" layer="19" extent="1-1"/>
-<wire x1="16.764" y1="6.628" x2="21.59" y2="6.628" width="0" layer="19" extent="1-1"/>
-<wire x1="15.748" y1="13.716" x2="16.764" y2="6.628" width="0" layer="19" extent="1-1"/>
-<wire x1="15.748" y1="16.256" x2="15.748" y2="13.716" width="0" layer="19" extent="1-1"/>
-<wire x1="9.144" y1="6.274" x2="16.764" y2="6.628" width="0" layer="19" extent="1-1"/>
-<wire x1="7.5692" y1="25.146" x2="15.748" y2="16.256" width="0" layer="19" extent="1-1"/>
-<wire x1="7.874" y1="30.226" x2="7.5692" y2="25.146" width="0" layer="19" extent="1-1"/>
-<wire x1="10.16" y1="34.798" x2="7.874" y2="30.226" width="0" layer="19" extent="1-1"/>
-<wire x1="7.366" y1="40.132" x2="10.16" y2="34.798" width="0" layer="19" extent="1-1"/>
-<wire x1="-25.4" y1="-8.89" x2="9.144" y2="6.274" width="0" layer="19" extent="1-1"/>
-<wire x1="-33.02" y1="-6.35" x2="-25.4" y2="-8.89" width="0" layer="19" extent="1-1"/>
+<wire x1="15.748" y1="13.716" x2="15.748" y2="16.256" width="0" layer="19" extent="1-1"/>
 </signal>
 <signal name="VCC">
@@
 <wire x1="57.404" y1="16.256" x2="57.658" y2="16.002" width="0.4064" layer="1"/>
 <wire x1="57.658" y1="16.002" x2="59.69" y2="18.034" width="0.4064" layer="1"/>
+<contactref element="R10" pad="1"/>
+<contactref element="R11" pad="2"/>
+<wire x1="44.45" y1="31.75" x2="41.91" y2="31.75" width="0.4064" layer="1"/>
+<wire x1="41.91" y1="31.75" x2="39.37" y2="34.29" width="0.4064" layer="1"/>
+<wire x1="52.832" y1="21.844" x2="52.832" y2="23.368" width="0.4064" layer="1"/>
+<wire x1="52.832" y1="23.368" x2="44.45" y2="31.75" width="0.4064" layer="1"/>
 </signal>
 <signal name="N$3">
@@
 <contactref element="R10" pad="2"/>
 <contactref element="JP7" pad="1"/>
-<wire x1="-16.51" y1="-5.08" x2="39.564" y2="21.971" width="0" layer="19" extent="1-1"/>
-<wire x1="-33.02" y1="-8.89" x2="-16.51" y2="-5.08" width="0" layer="19" extent="1-1"/>
+<wire x1="39.564" y1="21.971" x2="36.449" y2="21.971" width="0.4064" layer="1"/>
+<wire x1="36.449" y1="21.971" x2="35.56" y2="22.86" width="0.4064" layer="1"/>
+<wire x1="35.56" y1="22.86" x2="35.56" y2="26.67" width="0.4064" layer="1"/>
+<wire x1="35.56" y1="26.67" x2="38.1" y2="29.21" width="0.4064" layer="1"/>
+<wire x1="38.1" y1="29.21" x2="38.1" y2="35.56" width="0.4064" layer="1"/>
+<wire x1="38.1" y1="35.56" x2="39.37" y2="36.83" width="0.4064" layer="1"/>
+<wire x1="53.34" y1="31.75" x2="50.8" y2="31.75" width="0.4064" layer="1"/>
+<wire x1="50.8" y1="31.75" x2="45.72" y2="36.83" width="0.4064" layer="1"/>
+<wire x1="45.72" y1="36.83" x2="39.37" y2="36.83" width="0.4064" layer="1"/>
 </signal>
 <signal name="N$13">
 <contactref element="IC2" pad="6"/>
 <contactref element="R11" pad="1"/>
-<wire x1="-19.05" y1="-10.16" x2="39.564" y2="23.241" width="0" layer="19" extent="1-1"/>
-</signal>
-<signal name="N$14">
-<contactref element="R11" pad="2"/>
-<contactref element="R10" pad="1"/>
-<contactref element="JP3" pad="2"/>
-<wire x1="-19.05" y1="-5.08" x2="-25.4" y2="-6.35" width="0" layer="19" extent="1-1"/>
-<wire x1="-16.51" y1="-10.16" x2="-19.05" y2="-5.08" width="0" layer="19" extent="1-1"/>
+<wire x1="39.564" y1="23.241" x2="37.719" y2="23.241" width="0.4064" layer="1"/>
+<wire x1="37.719" y1="23.241" x2="36.83" y2="24.13" width="0.4064" layer="1"/>
+<wire x1="36.83" y1="24.13" x2="36.83" y2="25.4" width="0.4064" layer="1"/>
+<wire x1="36.83" y1="25.4" x2="40.64" y2="29.21" width="0.4064" layer="1"/>
+<wire x1="40.64" y1="29.21" x2="44.45" y2="29.21" width="0.4064" layer="1"/>
 </signal>
 </signals>

Commit message: test board included
Parts:
- moved C4 8.89 mm to (26.9, 7.87)
- moved C3 7.62 mm to (23.4, 7.87)
- moved C1 6.35 mm to (20.1, 8.13)
- moved C2 5.08 mm to (16.5, 8.13)
- moved C5 3.81 mm to (13.0, 8.13)
Routing:
- net VCC: track 81.4 -> 89.4 mm, vias 0 -> 1
Changed lines of the file:
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@@
 <?xml version="1.0" encoding="utf-8"?>
 <!DOCTYPE eagle SYSTEM "eagle.dtd">
-<eagle version="7.1.0">
+<eagle version="7.2.0">
 <drawing>
 <settings>
@@
 <setting verticaltext="up"/>
 </settings>
-<grid distance="0.05" unitdist="inch" unit="inch" style="lines" multiple="1" display="no" altdistance="0.025" altunitdist="inch" altunit="inch"/>
+<grid distance="0.05" unitdist="inch" unit="inch" style="lines" multiple="1" display="yes" altdistance="0.025" altunitdist="inch" altunit="inch"/>
 <layers>
 <layer number="1" name="Top" color="4" fill="1" visible="yes" active="yes"/>
@@
 <layer number="27" name="tValues" color="7" fill="1" visible="yes" active="yes"/>
 <layer number="28" name="bValues" color="7" fill="1" visible="yes" active="yes"/>
-<layer number="29" name="tStop" color="7" fill="3" visible="yes" active="yes"/>
-<layer number="30" name="bStop" color="7" fill="6" visible="yes" active="yes"/>
+<layer number="29" name="tStop" color="7" fill="3" visible="no" active="yes"/>
+<layer number="30" name="bStop" color="7" fill="6" visible="no" active="yes"/>
 <layer number="31" name="tCream" color="7" fill="4" visible="yes" active="yes"/>
 <layer number="32" name="bCream" color="7" fill="5" visible="yes" active="yes"/>
@@
 <element name="JP2" library="jumper" package="JP1" value="" x="60.96" y="18.034" rot="R90"/>
 <element name="USBMINI" library="adafruit" package="USB-MINIB" value="" x="5.08" y="7.874" rot="R270"/>
-<element name="C1" library="adafruit" package="C1206K" value="100uF" x="26.416" y="8.128" rot="R270"/>
-<element name="C2" library="adafruit" package="C1206K" value="10uF" x="21.59" y="8.128" rot="R270"/>
-<element name="C3" library="adafruit" package="C1206K" value="100uF" x="30.988" y="7.874" rot="R270"/>
-<element name="C4" library="adafruit" package="C1206K" value="100uF" x="35.814" y="7.874" rot="R270"/>
-<element name="C5" library="adafruit" package="C1206K" value="0.1uF" x="16.764" y="8.128" rot="R270"/>
+<element name="C1" library="adafruit" package="C1206K" value="100uF" x="20.066" y="8.128" rot="R270"/>
+<element name="C2" library="adafruit" package="C1206K" value="10uF" x="16.51" y="8.128" rot="R270"/>
+<element name="C3" library="adafruit" package="C1206K" value="100uF" x="23.368" y="7.874" rot="R270"/>
+<element name="C4" library="adafruit" package="C1206K" value="100uF" x="26.924" y="7.874" rot="R270"/>
+<element name="C5" library="adafruit" package="C1206K" value="0.1uF" x="12.954" y="8.128" rot="R270"/>
 <element name="JP4" library="jumper" package="JP1" value="" x="40.64" y="13.97" rot="R270"/>
 <element name="JP5" library="jumper" package="JP1" value="" x="33.02" y="29.718" rot="R270"/>
@@
 <contactref element="IC2" pad="5"/>
 <contactref element="JP7" pad="2"/>
+<via x="16.51" y="26.67" extent="1-16" drill="0.8"/>
 <wire x1="15.748" y1="13.716" x2="15.748" y2="16.256" width="0" layer="19" extent="1-1"/>
 </signal>
@@
 <contactref element="R6" pad="1"/>
 <wire x1="7.5692" y1="24.2062" x2="7.6454" y2="24.13" width="0.4064" layer="1"/>
-<wire x1="9.144" y1="9.474" x2="16.61" y2="9.474" width="0.4064" layer="1"/>
-<wire x1="16.61" y1="9.474" x2="16.764" y2="9.628" width="0.4064" layer="1"/>
-<wire x1="16.764" y1="9.628" x2="21.59" y2="9.628" width="0.4064" layer="1"/>
-<wire x1="21.59" y1="9.628" x2="23.876" y2="9.628" width="0.4064" layer="1"/>
-<wire x1="23.876" y1="9.628" x2="26.416" y2="9.628" width="0.4064" layer="1"/>
-<wire x1="26.416" y1="9.628" x2="30.734" y2="9.628" width="0.4064" layer="1"/>
-<wire x1="30.734" y1="9.628" x2="30.988" y2="9.374" width="0.4064" layer="1"/>
-<wire x1="30.988" y1="9.374" x2="35.814" y2="9.374" width="0.4064" layer="1"/>
-<wire x1="35.814" y1="9.374" x2="38.33" y2="9.374" width="0.4064" layer="1"/>
-<wire x1="38.33" y1="9.374" x2="39.37" y2="10.414" width="0.4064" layer="1"/>
-<wire x1="39.37" y1="10.414" x2="39.37" y2="13.97" width="0.4064" layer="1"/>
 <wire x1="39.37" y1="13.97" x2="39.37" y2="16.002" width="0.4064" layer="1"/>
 <wire x1="39.37" y1="16.002" x2="36.322" y2="19.05" width="0.4064" layer="1"/>
@@
 <wire x1="36.576" y1="20.574" x2="39.437" y2="20.574" width="0.4064" layer="1"/>
 <wire x1="39.437" y1="20.574" x2="39.564" y2="20.701" width="0.4064" layer="1"/>
-<wire x1="10.922" y1="24.13" x2="16.002" y2="24.13" width="0.4064" layer="1"/>
-<wire x1="16.002" y1="24.13" x2="16.256" y2="24.13" width="0.4064" layer="1"/>
-<wire x1="16.256" y1="24.13" x2="23.876" y2="16.51" width="0.4064" layer="1"/>
-<wire x1="23.876" y1="16.51" x2="23.876" y2="9.628" width="0.4064" layer="1"/>
-<wire x1="16.7386" y1="30.226" x2="16.7386" y2="24.8666" width="0.4064" layer="1"/>
-<wire x1="16.7386" y1="24.8666" x2="16.002" y2="24.13" width="0.4064" layer="1"/>
 <wire x1="7.6454" y1="24.13" x2="10.922" y2="24.13" width="0.4064" layer="1"/>
 <wire x1="5.1308" y1="26.0858" x2="5.6642" y2="26.0858" width="0.4064" layer="1"/>
@@
 <wire x1="6.35" y1="25.4" x2="7.5438" y2="24.2062" width="0.4064" layer="1" curve="90"/>
 <wire x1="7.5438" y1="24.2062" x2="7.5692" y2="24.2062" width="0.4064" layer="1"/>
+<wire x1="9.144" y1="9.474" x2="12.954" y2="9.474" width="0.4064" layer="1"/>
+<wire x1="12.954" y1="9.474" x2="12.954" y2="9.628" width="0.4064" layer="1"/>
+<wire x1="12.954" y1="9.628" x2="16.51" y2="9.628" width="0.4064" layer="1"/>
+<wire x1="16.51" y1="9.628" x2="20.066" y2="9.628" width="0.4064" layer="1"/>
+<wire x1="20.066" y1="9.628" x2="23.368" y2="9.628" width="0.4064" layer="1"/>
+<wire x1="23.368" y1="9.628" x2="23.368" y2="9.374" width="0.4064" layer="1"/>
+<wire x1="23.368" y1="9.374" x2="26.924" y2="9.374" width="0.4064" layer="1"/>
+<wire x1="26.924" y1="9.374" x2="34.774" y2="9.374" width="0.4064" layer="1"/>
+<wire x1="34.774" y1="9.374" x2="39.37" y2="13.97" width="0.4064" layer="1"/>
+<wire x1="10.922" y1="24.13" x2="15.24" y2="24.13" width="0.4064" layer="1"/>
+<via x="15.24" y="24.13" extent="1-16" drill="0.7"/>
+<wire x1="15.24" y1="24.13" x2="39.37" y2="13.97" width="0.4064" layer="16"/>
+<wire x1="16.7386" y1="30.226" x2="14.986" y2="30.226" width="0.4064" layer="1"/>
+<wire x1="14.986" y1="30.226" x2="13.97" y2="29.21" width="0.4064" layer="1"/>
+<wire x1="13.97" y1="29.21" x2="13.97" y2="25.4" width="0.4064" layer="1"/>
+<wire x1="13.97" y1="25.4" x2="15.24" y2="24.13" width="0.4064" layer="1"/>
 </signal>
 <signal name="N$4">
