File: Eagle/MSGP/MSGP.sch (EAGLE design)
At the start: 13 parts, among them T1 2N3904

Commit message: MSBP board
Parts:
- removed C6: (no value), rcl:C-US050-045X075
- added C7, C8: (no value), rcl:C-US050-045X075
- added R5: (no value), rcl:R-US_0207/10
Connections:
- removed net N$7: C6.1, U$1.CONT
- new net N$6: C5.1, U$1.THRES, U$1.TRIG
- new net N$9: C8.1, R5.2
- net GND: now also C7.2, C8.2; no longer C6.2
- net N$1: now also R5.1; no longer C5.1, U$1.THRES
- net VCC: now also C7.1, U$1.RESET
Other:
- moved on the sheet: R4
Changed lines of the file:
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@@
 <?xml version="1.0" encoding="utf-8"?>
 <!DOCTYPE eagle SYSTEM "eagle.dtd">
-<eagle version="7.1.0">
+<eagle version="7.2.0">
 <drawing>
 <settings>
@@
 <setting verticaltext="up"/>
 </settings>
-<grid distance="0.1" unitdist="inch" unit="inch" style="lines" multiple="1" display="yes" altdistance="0.01" altunitdist="inch" altunit="inch"/>
+<grid distance="0.1" unitdist="inch" unit="inch" style="lines" multiple="1" display="no" altdistance="0.01" altunitdist="inch" altunit="inch"/>
 <layers>
 <layer number="1" name="Top" color="4" fill="1" visible="no" active="no"/>
@@
 <part name="R4" library="rcl" deviceset="R-US_" device="0207/10"/>
 <part name="C5" library="rcl" deviceset="C-US" device="050-045X075"/>
-<part name="C6" library="rcl" deviceset="C-US" device="050-045X075"/>
+<part name="R5" library="rcl" deviceset="R-US_" device="0207/10"/>
+<part name="C7" library="rcl" deviceset="C-US" device="050-045X075"/>
+<part name="GND5" library="supply1" deviceset="GND" device=""/>
+<part name="C8" library="rcl" deviceset="C-US" device="050-045X075"/>
+<part name="GND6" library="supply1" deviceset="GND" device=""/>
 </parts>
 <sheets>
@@
 <instance part="GND4" gate="1" x="88.9" y="5.08"/>
 <instance part="P+2" gate="VCC" x="22.86" y="50.8"/>
-<instance part="R4" gate="G$1" x="12.7" y="45.72"/>
+<instance part="R4" gate="G$1" x="68.58" y="48.26" rot="R90"/>
 <instance part="C5" gate="G$1" x="12.7" y="22.86"/>
-<instance part="C6" gate="G$1" x="17.78" y="12.7"/>
+<instance part="R5" gate="G$1" x="68.58" y="33.02" rot="R270"/>
+<instance part="C7" gate="G$1" x="27.94" y="63.5"/>
+<instance part="GND5" gate="1" x="27.94" y="55.88"/>
+<instance part="C8" gate="G$1" x="68.58" y="22.86"/>
+<instance part="GND6" gate="1" x="68.58" y="15.24"/>
 </instances>
 <busses>
@@
 <pinref part="P+2" gate="VCC" pin="VCC"/>
 <wire x1="22.86" y1="43.18" x2="22.86" y2="45.72" width="0.1524" layer="91"/>
+<wire x1="22.86" y1="45.72" x2="22.86" y2="48.26" width="0.1524" layer="91"/>
+<wire x1="22.86" y1="45.72" x2="10.16" y2="45.72" width="0.1524" layer="91"/>
+<junction x="22.86" y="45.72"/>
+<wire x1="10.16" y1="45.72" x2="10.16" y2="66.04" width="0.1524" layer="91"/>
+<wire x1="10.16" y1="66.04" x2="27.94" y2="66.04" width="0.1524" layer="91"/>
 <pinref part="R4" gate="G$1" pin="2"/>
-<wire x1="22.86" y1="45.72" x2="22.86" y2="48.26" width="0.1524" layer="91"/>
-<wire x1="22.86" y1="45.72" x2="17.78" y2="45.72" width="0.1524" layer="91"/>
+<wire x1="27.94" y1="66.04" x2="68.58" y2="66.04" width="0.1524" layer="91"/>
+<wire x1="68.58" y1="66.04" x2="68.58" y2="53.34" width="0.1524" layer="91"/>
+<pinref part="C7" gate="G$1" pin="1"/>
+<junction x="27.94" y="66.04"/>
+</segment>
+<segment>
+<pinref part="U$1" gate="G$1" pin="RESET"/>
+<wire x1="22.86" y1="22.86" x2="20.32" y2="22.86" width="0.1524" layer="91"/>
+<label x="17.78" y="22.86" size="1.778" layer="95"/>
 </segment>
 </net>
@@
 <pinref part="C5" gate="G$1" pin="2"/>
 <wire x1="12.7" y1="17.78" x2="12.7" y2="7.62" width="0.1524" layer="91"/>
-<wire x1="12.7" y1="7.62" x2="17.78" y2="7.62" width="0.1524" layer="91"/>
-<pinref part="C6" gate="G$1" pin="2"/>
-<wire x1="17.78" y1="7.62" x2="22.86" y2="7.62" width="0.1524" layer="91"/>
-<junction x="17.78" y="7.62"/>
+<wire x1="12.7" y1="7.62" x2="22.86" y2="7.62" width="0.1524" layer="91"/>
 </segment>
 <segment>
@@
 <pinref part="C3" gate="G$1" pin="2"/>
 <pinref part="GND2" gate="1" pin="GND"/>
+</segment>
+<segment>
+<pinref part="C7" gate="G$1" pin="2"/>
+<pinref part="GND5" gate="1" pin="GND"/>
+</segment>
+<segment>
+<pinref part="C8" gate="G$1" pin="2"/>
+<pinref part="GND6" gate="1" pin="GND"/>
 </segment>
 </net>
@@
 <net name="N$1" class="0">
 <segment>
+<pinref part="U$1" gate="G$1" pin="DISCH"/>
+<pinref part="R4" gate="G$1" pin="1"/>
+<pinref part="R5" gate="G$1" pin="1"/>
+<wire x1="68.58" y1="43.18" x2="68.58" y2="40.64" width="0.1524" layer="91"/>
+<wire x1="68.58" y1="40.64" x2="68.58" y2="38.1" width="0.1524" layer="91"/>
+<wire x1="58.42" y1="40.64" x2="68.58" y2="40.64" width="0.1524" layer="91"/>
+<junction x="68.58" y="40.64"/>
+</segment>
+</net>
+<net name="N$6" class="0">
+<segment>
 <pinref part="U$1" gate="G$1" pin="THRES"/>
-<pinref part="R4" gate="G$1" pin="1"/>
-<wire x1="22.86" y1="27.94" x2="12.7" y2="27.94" width="0.1524" layer="91"/>
-<wire x1="12.7" y1="27.94" x2="7.62" y2="27.94" width="0.1524" layer="91"/>
-<wire x1="7.62" y1="27.94" x2="7.62" y2="45.72" width="0.1524" layer="91"/>
-<wire x1="7.62" y1="45.72" x2="7.62" y2="55.88" width="0.1524" layer="91"/>
-<wire x1="7.62" y1="55.88" x2="63.5" y2="55.88" width="0.1524" layer="91"/>
-<wire x1="63.5" y1="55.88" x2="63.5" y2="40.64" width="0.1524" layer="91"/>
-<pinref part="U$1" gate="G$1" pin="DISCH"/>
-<wire x1="63.5" y1="40.64" x2="58.42" y2="40.64" width="0.1524" layer="91"/>
+<wire x1="22.86" y1="27.94" x2="20.32" y2="27.94" width="0.1524" layer="91"/>
 <pinref part="C5" gate="G$1" pin="1"/>
+<wire x1="20.32" y1="27.94" x2="12.7" y2="27.94" width="0.1524" layer="91"/>
 <wire x1="12.7" y1="25.4" x2="12.7" y2="27.94" width="0.1524" layer="91"/>
-</segment>
-</net>
-<net name="N$7" class="0">
-<segment>
-<pinref part="U$1" gate="G$1" pin="CONT"/>
-<wire x1="22.86" y1="38.1" x2="17.78" y2="38.1" width="0.1524" layer="91"/>
-<wire x1="17.78" y1="38.1" x2="17.78" y2="15.24" width="0.1524" layer="91"/>
-<pinref part="C6" gate="G$1" pin="1"/>
-</segment>
-</net>
+<pinref part="U$1" gate="G$1" pin="TRIG"/>
+<wire x1="22.86" y1="33.02" x2="20.32" y2="33.02" width="0.1524" layer="91"/>
+<wire x1="20.32" y1="33.02" x2="20.32" y2="27.94" width="0.1524" layer="91"/>
+<junction x="20.32" y="27.94"/>
+</segment>
+</net>
+<net name="N$9" class="0">
+<segment>
+<pinref part="R5" gate="G$1" pin="2"/>
+<pinref part="C8" gate="G$1" pin="1"/>
+<wire x1="68.58" y1="27.94" x2="68.58" y2="25.4" width="0.1524" layer="91"/>
+</segment>
+</net>

Commit message: new MSGP
Parts:
- removed C1, C2, C3, C4, C5, C7, C8: (no value), rcl:C-US050-045X075
- removed L1: (no value), rcl:L-US0207/10
- removed R1, R2, R3, R4, R5: (no value), rcl:R-US_0207/10
- removed T1: 2N3904, transistor-neu-to92:2N3904
- removed U$1: LMC555, E3VB_ISI:LMC555
- added IC1: 74ALS04D, 74xx-us:74ALS04D
- added U1: LTC6905CS5TRMPBF, LTC_By_element14_Batch_1:LTC6905CS5TRMPBF
Connections:
- removed net GND: C1.2, C2.2, C3.2, C5.2, C7.2, C8.2, T1.E, U$1.GND
- removed net N$1: R4.1, R5.1, U$1.DISCH
- removed net N$2: C2.1, L1.2
- removed net N$3: C4.1, R1.2, R2.2, R3.1, T1.C
- removed net N$4: C3.1, C4.2, L1.1
- removed net N$5: C1.1, R1.1, R2.1, T1.B
- removed net N$6: C5.1, U$1.THRES, U$1.TRIG
- removed net N$9: C8.1, R5.2
- removed net VCC: C7.1, R3.2, R4.2, U$1.RESET, U$1.VDD
Changed lines of the file:
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@@
 </classes>
 <parts>
-<part name="U$1" library="E3VB_ISI" deviceset="LMC555" device=""/>
-<part name="R1" library="rcl" deviceset="R-US_" device="0207/10"/>
-<part name="C1" library="rcl" deviceset="C-US" device="050-045X075"/>
-<part name="C2" library="rcl" deviceset="C-US" device="050-045X075"/>
-<part name="C3" library="rcl" deviceset="C-US" device="050-045X075"/>
-<part name="L1" library="rcl" deviceset="L-US" device="0207/10"/>
-<part name="P+1" library="supply1" deviceset="VCC" device=""/>
-<part name="GND1" library="supply1" deviceset="GND" device=""/>
-<part name="T1" library="transistor-neu-to92" deviceset="2N3904" device=""/>
-<part name="R2" library="rcl" deviceset="R-US_" device="0207/10"/>
-<part name="GND2" library="supply1" deviceset="GND" device=""/>
-<part name="GND3" library="supply1" deviceset="GND" device=""/>
-<part name="R3" library="rcl" deviceset="R-US_" device="0207/10"/>
-<part name="C4" library="rcl" deviceset="C-US" device="050-045X075"/>
-<part name="GND4" library="supply1" deviceset="GND" device=""/>
-<part name="P+2" library="supply1" deviceset="VCC" device=""/>
-<part name="R4" library="rcl" deviceset="R-US_" device="0207/10"/>
-<part name="C5" library="rcl" deviceset="C-US" device="050-045X075"/>
-<part name="R5" library="rcl" deviceset="R-US_" device="0207/10"/>
-<part name="C7" library="rcl" deviceset="C-US" device="050-045X075"/>
-<part name="GND5" library="supply1" deviceset="GND" device=""/>
-<part name="C8" library="rcl" deviceset="C-US" device="050-045X075"/>
-<part name="GND6" library="supply1" deviceset="GND" device=""/>
+<part name="IC1" library="74xx-us" deviceset="74*04" device="D" technology="ALS"/>
+<part name="U1" library="LTC_By_element14_Batch_1" deviceset="LTC6905CS5TRMPBF" device=""/>
 </parts>
 <sheets>
@@
 </plain>
 <instances>
-<instance part="U$1" gate="G$1" x="40.64" y="30.48"/>
-<instance part="R1" gate="G$1" x="99.06" y="55.88"/>
-<instance part="C1" gate="G$1" x="88.9" y="20.32"/>
-<instance part="C2" gate="G$1" x="157.48" y="33.02"/>
-<instance part="C3" gate="G$1" x="139.7" y="33.02"/>
-<instance part="L1" gate="G$1" x="149.86" y="35.56" rot="R90"/>
-<instance part="P+1" gate="VCC" x="119.38" y="53.34"/>
-<instance part="GND1" gate="1" x="106.68" y="22.86"/>
-<instance part="T1" gate="G1" x="104.14" y="30.48"/>
-<instance part="R2" gate="G$1" x="99.06" y="48.26"/>
-<instance part="GND2" gate="1" x="139.7" y="25.4"/>
-<instance part="GND3" gate="1" x="157.48" y="25.4"/>
-<instance part="R3" gate="G$1" x="119.38" y="43.18" rot="R90"/>
-<instance part="C4" gate="G$1" x="129.54" y="35.56" rot="R90"/>
-<instance part="GND4" gate="1" x="88.9" y="5.08"/>
-<instance part="P+2" gate="VCC" x="22.86" y="50.8"/>
-<instance part="R4" gate="G$1" x="68.58" y="48.26" rot="R90"/>
-<instance part="C5" gate="G$1" x="12.7" y="22.86"/>
-<instance part="R5" gate="G$1" x="68.58" y="33.02" rot="R270"/>
-<instance part="C7" gate="G$1" x="27.94" y="63.5"/>
-<instance part="GND5" gate="1" x="27.94" y="55.88"/>
-<instance part="C8" gate="G$1" x="68.58" y="22.86"/>
-<instance part="GND6" gate="1" x="68.58" y="15.24"/>
+<instance part="IC1" gate="A" x="60.96" y="48.26"/>
+<instance part="IC1" gate="B" x="60.96" y="30.48"/>
+<instance part="IC1" gate="C" x="101.6" y="53.34"/>
+<instance part="IC1" gate="D" x="99.06" y="33.02"/>
+<instance part="IC1" gate="P" x="35.56" y="58.42"/>
+<instance part="IC1" gate="E" x="137.16" y="53.34"/>
+<instance part="IC1" gate="F" x="137.16" y="33.02"/>
+<instance part="U1" gate="A" x="78.74" y="71.12"/>
 </instances>
 <busses>
 </busses>
 <nets>
-<net name="VCC" class="0">
-<segment>
-<pinref part="P+1" gate="VCC" pin="VCC"/>
-<pinref part="R3" gate="G$1" pin="2"/>
-<wire x1="119.38" y1="50.8" x2="119.38" y2="48.26" width="0.1524" layer="91"/>
-</segment>
-<segment>
-<pinref part="U$1" gate="G$1" pin="VDD"/>
-<pinref part="P+2" gate="VCC" pin="VCC"/>
-<wire x1="22.86" y1="43.18" x2="22.86" y2="45.72" width="0.1524" layer="91"/>
-<wire x1="22.86" y1="45.72" x2="22.86" y2="48.26" width="0.1524" layer="91"/>
-<wire x1="22.86" y1="45.72" x2="10.16" y2="45.72" width="0.1524" layer="91"/>
-<junction x="22.86" y="45.72"/>
-<wire x1="10.16" y1="45.72" x2="10.16" y2="66.04" width="0.1524" layer="91"/>
-<wire x1="10.16" y1="66.04" x2="27.94" y2="66.04" width="0.1524" layer="91"/>
-<pinref part="R4" gate="G$1" pin="2"/>
-<wire x1="27.94" y1="66.04" x2="68.58" y2="66.04" width="0.1524" layer="91"/>
-<wire x1="68.58" y1="66.04" x2="68.58" y2="53.34" width="0.1524" layer="91"/>
-<pinref part="C7" gate="G$1" pin="1"/>
-<junction x="27.94" y="66.04"/>
-</segment>
-<segment>
-<pinref part="U$1" gate="G$1" pin="RESET"/>
-<wire x1="22.86" y1="22.86" x2="20.32" y2="22.86" width="0.1524" layer="91"/>
-<label x="17.78" y="22.86" size="1.778" layer="95"/>
-</segment>
-</net>
-<net name="N$2" class="0">
-<segment>
-<pinref part="C2" gate="G$1" pin="1"/>
-<pinref part="L1" gate="G$1" pin="2"/>
-</segment>
-</net>
-<net name="N$3" class="0">
-<segment>
-<pinref part="R3" gate="G$1" pin="1"/>
-<wire x1="119.38" y1="35.56" x2="119.38" y2="38.1" width="0.1524" layer="91"/>
-<pinref part="T1" gate="G1" pin="C"/>
-<wire x1="109.22" y1="35.56" x2="109.22" y2="48.26" width="0.1524" layer="91"/>
-<wire x1="109.22" y1="48.26" x2="109.22" y2="55.88" width="0.1524" layer="91"/>
-<wire x1="109.22" y1="35.56" x2="106.68" y2="35.56" width="0.1524" layer="91"/>
-<pinref part="R2" gate="G$1" pin="2"/>
-<wire x1="104.14" y1="48.26" x2="109.22" y2="48.26" width="0.1524" layer="91"/>
-<pinref part="R1" gate="G$1" pin="2"/>
-<wire x1="104.14" y1="55.88" x2="109.22" y2="55.88" width="0.1524" layer="91"/>
-<pinref part="C4" gate="G$1" pin="1"/>
-<wire x1="127" y1="35.56" x2="119.38" y2="35.56" width="0.1524" layer="91"/>
-<junction x="119.38" y="35.56"/>
-<wire x1="119.38" y1="35.56" x2="109.22" y2="35.56" width="0.1524" layer="91"/>
-</segment>
-</net>
-<net name="GND" class="0">
-<segment>
-<pinref part="GND4" gate="1" pin="GND"/>
-<pinref part="U$1" gate="G$1" pin="GND"/>
-<wire x1="22.86" y1="17.78" x2="22.86" y2="7.62" width="0.1524" layer="91"/>
-<wire x1="22.86" y1="7.62" x2="88.9" y2="7.62" width="0.1524" layer="91"/>
-<pinref part="C1" gate="G$1" pin="2"/>
-<wire x1="88.9" y1="7.62" x2="88.9" y2="15.24" width="0.1524" layer="91"/>
-<pinref part="C5" gate="G$1" pin="2"/>
-<wire x1="12.7" y1="17.78" x2="12.7" y2="7.62" width="0.1524" layer="91"/>
-<wire x1="12.7" y1="7.62" x2="22.86" y2="7.62" width="0.1524" layer="91"/>
-</segment>
-<segment>
-<pinref part="T1" gate="G1" pin="E"/>
-<pinref part="GND1" gate="1" pin="GND"/>
-</segment>
-<segment>
-<pinref part="C2" gate="G$1" pin="2"/>
-<pinref part="GND3" gate="1" pin="GND"/>
-</segment>
-<segment>
-<pinref part="C3" gate="G$1" pin="2"/>
-<pinref part="GND2" gate="1" pin="GND"/>
-</segment>
-<segment>
-<pinref part="C7" gate="G$1" pin="2"/>
-<pinref part="GND5" gate="1" pin="GND"/>
-</segment>
-<segment>
-<pinref part="C8" gate="G$1" pin="2"/>
-<pinref part="GND6" gate="1" pin="GND"/>
-</segment>
-</net>
-<net name="N$5" class="0">
-<segment>
-<pinref part="T1" gate="G1" pin="B"/>
-<wire x1="101.6" y1="30.48" x2="88.9" y2="30.48" width="0.1524" layer="91"/>
-<pinref part="R1" gate="G$1" pin="1"/>
-<wire x1="93.98" y1="55.88" x2="88.9" y2="55.88" width="0.1524" layer="91"/>
-<wire x1="88.9" y1="55.88" x2="88.9" y2="48.26" width="0.1524" layer="91"/>
-<pinref part="R2" gate="G$1" pin="1"/>
-<wire x1="93.98" y1="48.26" x2="88.9" y2="48.26" width="0.1524" layer="91"/>
-<wire x1="88.9" y1="48.26" x2="88.9" y2="30.48" width="0.1524" layer="91"/>
-<pinref part="C1" gate="G$1" pin="1"/>
-<wire x1="88.9" y1="22.86" x2="88.9" y2="30.48" width="0.1524" layer="91"/>
-</segment>
-</net>
-<net name="N$4" class="0">
-<segment>
-<pinref part="C3" gate="G$1" pin="1"/>
-<pinref part="L1" gate="G$1" pin="1"/>
-<wire x1="142.24" y1="35.56" x2="139.7" y2="35.56" width="0.1524" layer="91"/>
-<pinref part="C4" gate="G$1" pin="2"/>
-<wire x1="139.7" y1="35.56" x2="134.62" y2="35.56" width="0.1524" layer="91"/>
-</segment>
-</net>
-<net name="N$1" class="0">
-<segment>
-<pinref part="U$1" gate="G$1" pin="DISCH"/>
-<pinref part="R4" gate="G$1" pin="1"/>
-<pinref part="R5" gate="G$1" pin="1"/>
-<wire x1="68.58" y1="43.18" x2="68.58" y2="40.64" width="0.1524" layer="91"/>
-<wire x1="68.58" y1="40.64" x2="68.58" y2="38.1" width="0.1524" layer="91"/>
-<wire x1="58.42" y1="40.64" x2="68.58" y2="40.64" width="0.1524" layer="91"/>
-<junction x="68.58" y="40.64"/>
-</segment>
-</net>
-<net name="N$6" class="0">
-<segment>
-<pinref part="U$1" gate="G$1" pin="THRES"/>
-<wire x1="22.86" y1="27.94" x2="20.32" y2="27.94" width="0.1524" layer="91"/>
-<pinref part="C5" gate="G$1" pin="1"/>
-<wire x1="20.32" y1="27.94" x2="12.7" y2="27.94" width="0.1524" layer="91"/>
-<wire x1="12.7" y1="25.4" x2="12.7" y2="27.94" width="0.1524" layer="91"/>
-<pinref part="U$1" gate="G$1" pin="TRIG"/>
-<wire x1="22.86" y1="33.02" x2="20.32" y2="33.02" width="0.1524" layer="91"/>
-<wire x1="20.32" y1="33.02" x2="20.32" y2="27.94" width="0.1524" layer="91"/>
-<junction x="20.32" y="27.94"/>
-</segment>
-</net>
-<net name="N$9" class="0">
-<segment>
-<pinref part="R5" gate="G$1" pin="2"/>
-<pinref part="C8" gate="G$1" pin="1"/>
-<wire x1="68.58" y1="27.94" x2="68.58" y2="25.4" width="0.1524" layer="91"/>
-</segment>
-</net>
 </nets>
 </sheet>
