File: Eagle/MSGP/MSGP.sch (EAGLE design)
At the start: 18 parts, among them IC1 74ALS04D, IC2 NE5532D, U1 LTC6905CS5TRMPBF

Commit message: MSG layout
Parts:
- removed JP3: (no value), jumper:JP1E
- added R4, R5, R6, R7, R8, R9: (no value), resistor:R-US_0204/2V
- R1, R2, R3: device rcl:R-US_R0805 -> resistor:R-US_0204/2V
Connections:
- new net N$10: IC1C.O, R7.1
- new net N$11: IC1F.O, R9.1
- new net N$7: IC1A.O, R1.1
- new net N$8: IC1B.O, R2.1
- new net N$9: IC1D.O, R3.1
- net GND: now also R1.2, R2.2, R3.2, R7.2, R8.2, R9.2; no longer JP3.2
- net N$2: now also R4.1, R5.1; no longer R1.1, R2.1
- net N$3: now also R5.2; no longer R1.2
- net N$4: now also R8.1; no longer IC1A.O, IC1B.O, IC1C.O, IC1D.O, IC1F.O, JP3.1
- net N$5: now also R4.2; no longer R2.2
- net N$6: now also R6.2; no longer R3.1
- net VCC: now also R6.1; no longer R3.2
Other:
- moved on the sheet: R1, R2, R3

Commit message: Schem
Parts:
- added JP3, JP7: (no value), jumper:JP1E
- added R10, R11: (no value), resistor:R-US_0204/2V
Connections:
- new net N$12: IC2B.OUT, JP7.1, R10.2
- new net N$13: IC2B.-IN, R11.1
- new net N$14: JP3.2, R10.1, R11.2
- net GND: now also IC2B.+IN, JP3.1, JP7.2
Other:
- moved on the sheet: JP5, JP6
Changed lines of the file:
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@@
 <part name="GND22" library="supply1" deviceset="GND" device=""/>
 <part name="GND23" library="supply1" deviceset="GND" device=""/>
+<part name="R10" library="resistor" deviceset="R-US_" device="0204/2V"/>
+<part name="R11" library="resistor" deviceset="R-US_" device="0204/2V"/>
+<part name="GND24" library="supply1" deviceset="GND" device=""/>
+<part name="JP3" library="jumper" deviceset="JP1E" device=""/>
+<part name="GND25" library="supply1" deviceset="GND" device=""/>
+<part name="JP7" library="jumper" deviceset="JP1E" device=""/>
+<part name="GND26" library="supply1" deviceset="GND" device=""/>
 </parts>
 <sheets>
@@
 <instance part="GND21" gate="1" x="-58.42" y="76.2"/>
 <instance part="JP4" gate="A" x="-45.72" y="81.28" rot="R270"/>
-<instance part="JP5" gate="A" x="-33.02" y="-7.62"/>
-<instance part="JP6" gate="A" x="-17.78" y="-7.62"/>
-<instance part="GND13" gate="1" x="-38.1" y="-12.7"/>
-<instance part="GND14" gate="1" x="-27.94" y="-12.7"/>
-<instance part="GND15" gate="1" x="-17.78" y="-15.24"/>
-<instance part="GND16" gate="1" x="-10.16" y="-15.24"/>
+<instance part="JP5" gate="A" x="-38.1" y="-20.32"/>
+<instance part="JP6" gate="A" x="-15.24" y="-17.78"/>
+<instance part="GND13" gate="1" x="-43.18" y="-25.4"/>
+<instance part="GND14" gate="1" x="-30.48" y="-25.4"/>
+<instance part="GND15" gate="1" x="-17.78" y="-25.4"/>
+<instance part="GND16" gate="1" x="-10.16" y="-25.4"/>
 <instance part="R4" gate="G$1" x="-45.72" y="22.86"/>
 <instance part="R5" gate="G$1" x="-30.48" y="40.64"/>
@@
 <instance part="GND22" gate="1" x="114.3" y="-2.54" rot="R90"/>
 <instance part="GND23" gate="1" x="114.3" y="-15.24" rot="R90"/>
+<instance part="IC2" gate="B" x="-30.48" y="5.08"/>
+<instance part="R10" gate="G$1" x="-12.7" y="0" rot="R90"/>
+<instance part="R11" gate="G$1" x="-50.8" y="2.54" rot="R180"/>
+<instance part="GND24" gate="1" x="-45.72" y="7.62" rot="R270"/>
+<instance part="JP3" gate="A" x="-66.04" y="5.08"/>
+<instance part="GND25" gate="1" x="-66.04" y="0"/>
+<instance part="JP7" gate="A" x="-2.54" y="7.62"/>
+<instance part="GND26" gate="1" x="0" y="2.54"/>
 </instances>
 <busses>
@@
 <pinref part="JP5" gate="A" pin="1"/>
 <pinref part="GND13" gate="1" pin="GND"/>
-<wire x1="-33.02" y1="-10.16" x2="-38.1" y2="-10.16" width="0.1524" layer="91"/>
+<wire x1="-38.1" y1="-22.86" x2="-43.18" y2="-22.86" width="0.1524" layer="91"/>
 </segment>
 <segment>
 <pinref part="JP5" gate="A" pin="2"/>
 <pinref part="GND14" gate="1" pin="GND"/>
-<wire x1="-30.48" y1="-10.16" x2="-27.94" y2="-10.16" width="0.1524" layer="91"/>
+<wire x1="-35.56" y1="-22.86" x2="-30.48" y2="-22.86" width="0.1524" layer="91"/>
 </segment>
 <segment>
 <pinref part="JP6" gate="A" pin="1"/>
 <pinref part="GND15" gate="1" pin="GND"/>
-<wire x1="-17.78" y1="-10.16" x2="-17.78" y2="-12.7" width="0.1524" layer="91"/>
+<wire x1="-15.24" y1="-20.32" x2="-17.78" y2="-22.86" width="0.1524" layer="91"/>
 </segment>
 <segment>
 <pinref part="JP6" gate="A" pin="2"/>
-<wire x1="-15.24" y1="-10.16" x2="-15.24" y2="-12.7" width="0.1524" layer="91"/>
 <pinref part="GND16" gate="1" pin="GND"/>
-<wire x1="-15.24" y1="-12.7" x2="-10.16" y2="-12.7" width="0.1524" layer="91"/>
+<wire x1="-12.7" y1="-20.32" x2="-10.16" y2="-22.86" width="0.1524" layer="91"/>
 </segment>
 <segment>
@@
 <pinref part="GND23" gate="1" pin="GND"/>
 <junction x="111.76" y="-15.24"/>
+</segment>
+<segment>
+<pinref part="IC2" gate="B" pin="+IN"/>
+<pinref part="GND24" gate="1" pin="GND"/>
+<wire x1="-38.1" y1="7.62" x2="-43.18" y2="7.62" width="0.1524" layer="91"/>
+</segment>
+<segment>
+<pinref part="JP3" gate="A" pin="1"/>
+<pinref part="GND25" gate="1" pin="GND"/>
+</segment>
+<segment>
+<pinref part="JP7" gate="A" pin="2"/>
+<pinref part="GND26" gate="1" pin="GND"/>
 </segment>
 </net>
@@
 </segment>
 </net>
+<net name="N$12" class="0">
+<segment>
+<pinref part="IC2" gate="B" pin="OUT"/>
+<pinref part="R10" gate="G$1" pin="2"/>
+<wire x1="-22.86" y1="5.08" x2="-12.7" y2="5.08" width="0.1524" layer="91"/>
+<wire x1="-12.7" y1="5.08" x2="-2.54" y2="5.08" width="0.1524" layer="91"/>
+<pinref part="JP7" gate="A" pin="1"/>
+</segment>
+</net>
+<net name="N$13" class="0">
+<segment>
+<pinref part="IC2" gate="B" pin="-IN"/>
+<pinref part="R11" gate="G$1" pin="1"/>
+<wire x1="-38.1" y1="2.54" x2="-45.72" y2="2.54" width="0.1524" layer="91"/>
+</segment>
+</net>
+<net name="N$14" class="0">
+<segment>
+<pinref part="R11" gate="G$1" pin="2"/>
+<wire x1="-55.88" y1="2.54" x2="-55.88" y2="-5.08" width="0.1524" layer="91"/>
+<pinref part="R10" gate="G$1" pin="1"/>
+<wire x1="-55.88" y1="-5.08" x2="-12.7" y2="-5.08" width="0.1524" layer="91"/>
+<wire x1="-55.88" y1="2.54" x2="-63.5" y2="2.54" width="0.1524" layer="91"/>
+<pinref part="JP3" gate="A" pin="2"/>
+</segment>
+</net>

Commit message: Updated Schematic
Parts:
- removed JP3: (no value), jumper:JP1E
Connections:
- removed net N$14: JP3.2, R10.1, R11.2
- net GND: no longer JP3.1
- net N$2: now also R10.1, R11.2
Changed lines of the file:
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@@
 <part name="R11" library="resistor" deviceset="R-US_" device="0204/2V"/>
 <part name="GND24" library="supply1" deviceset="GND" device=""/>
-<part name="JP3" library="jumper" deviceset="JP1E" device=""/>
-<part name="GND25" library="supply1" deviceset="GND" device=""/>
 <part name="JP7" library="jumper" deviceset="JP1E" device=""/>
 <part name="GND26" library="supply1" deviceset="GND" device=""/>
@@
 <instance part="R11" gate="G$1" x="-50.8" y="2.54" rot="R180"/>
 <instance part="GND24" gate="1" x="-45.72" y="7.62" rot="R270"/>
-<instance part="JP3" gate="A" x="-66.04" y="5.08"/>
-<instance part="GND25" gate="1" x="-66.04" y="0"/>
 <instance part="JP7" gate="A" x="-2.54" y="7.62"/>
 <instance part="GND26" gate="1" x="0" y="2.54"/>
@@
 <pinref part="GND24" gate="1" pin="GND"/>
 <wire x1="-38.1" y1="7.62" x2="-43.18" y2="7.62" width="0.1524" layer="91"/>
-</segment>
-<segment>
-<pinref part="JP3" gate="A" pin="1"/>
-<pinref part="GND25" gate="1" pin="GND"/>
+<junction x="-43.18" y="7.62"/>
 </segment>
 <segment>
@@
 <wire x1="-50.8" y1="40.64" x2="-35.56" y2="40.64" width="0.1524" layer="91"/>
 <pinref part="JP2" gate="A" pin="2"/>
-<wire x1="-50.8" y1="22.86" x2="-58.42" y2="22.86" width="0.1524" layer="91"/>
+<wire x1="-50.8" y1="22.86" x2="-55.88" y2="22.86" width="0.1524" layer="91"/>
 <pinref part="R4" gate="G$1" pin="1"/>
 <junction x="-50.8" y="22.86"/>
 <pinref part="R5" gate="G$1" pin="1"/>
 <junction x="-35.56" y="40.64"/>
+<pinref part="R11" gate="G$1" pin="2"/>
+<wire x1="-55.88" y1="22.86" x2="-58.42" y2="22.86" width="0.1524" layer="91"/>
+<wire x1="-55.88" y1="2.54" x2="-55.88" y2="-5.08" width="0.1524" layer="91"/>
+<pinref part="R10" gate="G$1" pin="1"/>
+<wire x1="-55.88" y1="-5.08" x2="-12.7" y2="-5.08" width="0.1524" layer="91"/>
+<wire x1="-55.88" y1="22.86" x2="-55.88" y2="2.54" width="0.1524" layer="91"/>
+<junction x="-55.88" y="2.54"/>
+<junction x="-55.88" y="22.86"/>
+<junction x="-12.7" y="-5.08"/>
 </segment>
 </net>
@@
 <wire x1="-12.7" y1="5.08" x2="-2.54" y2="5.08" width="0.1524" layer="91"/>
 <pinref part="JP7" gate="A" pin="1"/>
+<junction x="-12.7" y="5.08"/>
+<junction x="-2.54" y="5.08"/>
 </segment>
 </net>
@@
 <pinref part="R11" gate="G$1" pin="1"/>
 <wire x1="-38.1" y1="2.54" x2="-45.72" y2="2.54" width="0.1524" layer="91"/>
-</segment>
-</net>
-<net name="N$14" class="0">
-<segment>
-<pinref part="R11" gate="G$1" pin="2"/>
-<wire x1="-55.88" y1="2.54" x2="-55.88" y2="-5.08" width="0.1524" layer="91"/>
-<pinref part="R10" gate="G$1" pin="1"/>
-<wire x1="-55.88" y1="-5.08" x2="-12.7" y2="-5.08" width="0.1524" layer="91"/>
-<wire x1="-55.88" y1="2.54" x2="-63.5" y2="2.54" width="0.1524" layer="91"/>
-<pinref part="JP3" gate="A" pin="2"/>
-</segment>
-</net>
+<junction x="-45.72" y="2.54"/>
+</segment>
+</net>

Commit message: some clean up
Parts:
- added IC3, IC4: 74ALS04D, 74xx-us:74ALS04D
- added JP10, JP12, JP13, JP3, JP8, JP9: (no value), jumper:JP1E
- added R12, R13, R14, R15, R16, R17, R18, R19: (no value), resistor:R-US_0204/2V
Connections:
- new net N$14: IC3E.O, R12.1
- new net N$16: IC3A.O, R4.1
- new net N$17: IC3B.O, R5.1
- new net N$18: IC3D.O, R10.1
- new net N$19: IC3C.O, R11.1
- new net N$20: IC3F.O, R13.1
- new net N$21: IC4E.O, R18.1
- new net N$23: IC4A.O, R14.1
- new net N$24: IC4B.O, R15.1
- new net N$25: IC4D.O, R16.1
- new net N$26: IC4C.O, R17.1
- new net N$27: IC4F.O, R19.1
- net GND: now also C1.2, IC3P.GND, IC4P.GND, JP13.2, R10.2, R11.2, R12.2, R13.2, R14.2, R15.2, R16.2, R17.2, R18.2, R19.2, R4.2, R5.2
- net N$1: now also IC3A.I, IC3B.I, IC3C.I, IC3D.I, IC3E.I, IC3F.I, IC4A.I, IC4B.I, IC4C.I, IC4D.I, IC4E.I, IC4F.I
- net N$12: now also JP8.2; no longer R10.2
- net N$13: now also JP3.2; no longer R11.1
- net N$2: now also JP10.1, JP3.1, JP8.1, JP9.1; no longer R10.1, R11.2, R4.1, R5.1
- net N$3: now also JP9.2; no longer R5.2
- net N$5: now also JP10.2; no longer R4.2
- net VCC: now also IC3P.VCC, IC4P.VCC, JP12.1, JP12.2, JP13.1
Other:
- moved on the sheet: IC1A, IC1B, IC1C, IC1D, IC1E, IC1F, IC2A, IC2B, JP1, JP2, JP5, JP6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
