File: Eagle/MSGP/MSGP_rev2.sch (EAGLE design)
At the start: 45 parts, among them IC1 74ALS04D, IC2 NE5532D, IC3 74ALS04D, IC4 74ALS04D, U1 LTC6905CS5TRMPBF

Commit message: updated boards
fixed some of the issued we encountered while making the board
Connections:
- removed net GND: C1.2, C2.2, C3.2, C4.2, C5.2, IC1P.GND, IC2A.+IN, IC2B.+IN, IC2P.V-, IC3P.GND, IC4P.GND, JP1.2, JP13.2, JP2.1, JP4.2, JP5.1, JP5.2, JP6.1, JP6.2, JP7.2, R1.2, R10.2, R11.2, R12.2, R13.2, R14.2, R15.2, R16.2, R17.2, R18.2, R19.2, R2.2, R3.2, R4.2, R5.2, R7.2, R8.2, R9.2, U1.GND, USBMINI.GND
- new net GNDA: C1.2, C2.2, C3.2, C4.2, C5.2, IC2A.+IN, IC2B.+IN, IC2P.V-, JP1.2, JP13.2, JP2.1, JP4.2, JP5.2, JP6.2, JP7.2, U1.GND, USBMINI.GND
- new net GND_D: IC1P.GND, IC3P.GND, IC4P.GND, JP5.1, JP6.1, R1.2, R10.2, R11.2, R12.2, R13.2, R14.2, R15.2, R16.2, R17.2, R18.2, R19.2, R2.2, R3.2, R4.2, R5.2, R7.2, R8.2, R9.2

Commit message: minor changes to MSGP rev2
change one trace to digital ground
Connections:
- removed net N$13: IC2B.-IN, JP3.2
- new net N$30: JP10.1, JP2.2, JP3.1
- net GNDA: no longer U1.GND
- net GND_D: now also U1.GND
- net N$2: now also IC2B.-IN, JP3.2; no longer JP10.1, JP2.2, JP3.1, JP9.1
- net N$5: now also JP9.1
Other:
- moved on the sheet: JP9
Changed lines of the file:
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@@
 <instance part="JP3" gate="A" x="-81.28" y="15.24"/>
 <instance part="JP8" gate="A" x="-40.64" y="10.16" rot="R90"/>
-<instance part="JP9" gate="A" x="-60.96" y="53.34"/>
+<instance part="JP9" gate="A" x="-55.88" y="27.94"/>
 <instance part="JP10" gate="A" x="-73.66" y="30.48"/>
 <instance part="IC3" gate="A" x="17.78" y="30.48"/>
@@
 <net name="N$2" class="0">
 <segment>
-<wire x1="-78.74" y1="33.02" x2="-78.74" y2="50.8" width="0.1524" layer="91"/>
-<wire x1="-78.74" y1="50.8" x2="-60.96" y2="50.8" width="0.1524" layer="91"/>
-<pinref part="JP2" gate="A" pin="2"/>
-<wire x1="-78.74" y1="33.02" x2="-83.82" y2="33.02" width="0.1524" layer="91"/>
-<wire x1="-83.82" y1="33.02" x2="-86.36" y2="33.02" width="0.1524" layer="91"/>
-<wire x1="-83.82" y1="5.08" x2="-38.1" y2="5.08" width="0.1524" layer="91"/>
-<wire x1="-83.82" y1="33.02" x2="-83.82" y2="12.7" width="0.1524" layer="91"/>
-<junction x="-83.82" y="33.02"/>
-<pinref part="JP9" gate="A" pin="1"/>
-<wire x1="-83.82" y1="12.7" x2="-83.82" y2="5.08" width="0.1524" layer="91"/>
-<wire x1="-78.74" y1="33.02" x2="-78.74" y2="27.94" width="0.1524" layer="91"/>
-<pinref part="JP10" gate="A" pin="1"/>
-<wire x1="-78.74" y1="27.94" x2="-73.66" y2="27.94" width="0.1524" layer="91"/>
-<pinref part="JP3" gate="A" pin="1"/>
-<wire x1="-81.28" y1="12.7" x2="-83.82" y2="12.7" width="0.1524" layer="91"/>
 <pinref part="JP8" gate="A" pin="1"/>
 <wire x1="-38.1" y1="10.16" x2="-38.1" y2="5.08" width="0.1524" layer="91"/>
-<junction x="-83.82" y="12.7"/>
-<junction x="-78.74" y="33.02"/>
+<pinref part="IC2" gate="B" pin="-IN"/>
+<wire x1="-66.04" y1="12.7" x2="-71.12" y2="12.7" width="0.1524" layer="91"/>
+<pinref part="JP3" gate="A" pin="2"/>
+<wire x1="-71.12" y1="12.7" x2="-78.74" y2="12.7" width="0.1524" layer="91"/>
+<wire x1="-38.1" y1="5.08" x2="-71.12" y2="5.08" width="0.1524" layer="91"/>
+<wire x1="-71.12" y1="5.08" x2="-71.12" y2="12.7" width="0.1524" layer="91"/>
+<junction x="-71.12" y="12.7"/>
 </segment>
 </net>
 <net name="N$3" class="0">
 <segment>
-<wire x1="-58.42" y1="50.8" x2="-38.1" y2="50.8" width="0.1524" layer="91"/>
-<wire x1="-38.1" y1="50.8" x2="-38.1" y2="35.56" width="0.1524" layer="91"/>
 <pinref part="IC2" gate="A" pin="OUT"/>
-<wire x1="-38.1" y1="35.56" x2="-45.72" y2="35.56" width="0.1524" layer="91"/>
 <pinref part="JP1" gate="A" pin="1"/>
 <wire x1="-30.48" y1="35.56" x2="-38.1" y2="35.56" width="0.1524" layer="91"/>
+<wire x1="-38.1" y1="35.56" x2="-45.72" y2="35.56" width="0.1524" layer="91"/>
+<wire x1="-38.1" y1="35.56" x2="-38.1" y2="25.4" width="0.1524" layer="91"/>
 <junction x="-38.1" y="35.56"/>
 <pinref part="JP9" gate="A" pin="2"/>
+<wire x1="-38.1" y1="25.4" x2="-53.34" y2="25.4" width="0.1524" layer="91"/>
 </segment>
 </net>
@@
 <segment>
 <pinref part="IC2" gate="A" pin="-IN"/>
-<wire x1="-60.96" y1="33.02" x2="-68.58" y2="33.02" width="0.1524" layer="91"/>
+<wire x1="-60.96" y1="33.02" x2="-63.5" y2="33.02" width="0.1524" layer="91"/>
 <pinref part="JP10" gate="A" pin="2"/>
+<wire x1="-63.5" y1="33.02" x2="-68.58" y2="33.02" width="0.1524" layer="91"/>
 <wire x1="-71.12" y1="27.94" x2="-68.58" y2="27.94" width="0.1524" layer="91"/>
 <wire x1="-68.58" y1="27.94" x2="-68.58" y2="33.02" width="0.1524" layer="91"/>
+<pinref part="JP9" gate="A" pin="1"/>
+<wire x1="-55.88" y1="25.4" x2="-63.5" y2="25.4" width="0.1524" layer="91"/>
+<wire x1="-63.5" y1="25.4" x2="-63.5" y2="33.02" width="0.1524" layer="91"/>
+<junction x="-63.5" y="33.02"/>
 </segment>
 </net>
@@
 <wire x1="-38.1" y1="12.7" x2="-38.1" y2="15.24" width="0.1524" layer="91"/>
 <junction x="-38.1" y="15.24"/>
-</segment>
-</net>
-<net name="N$13" class="0">
-<segment>
-<pinref part="IC2" gate="B" pin="-IN"/>
-<wire x1="-66.04" y1="12.7" x2="-78.74" y2="12.7" width="0.1524" layer="91"/>
-<pinref part="JP3" gate="A" pin="2"/>
 </segment>
 </net>
@@
 <wire x1="-60.96" y1="38.1" x2="-68.58" y2="38.1" width="0.1524" layer="91"/>
 </segment>
-<segment>
-<pinref part="U1" gate="A" pin="GND"/>
-<pinref part="GND1" gate="1" pin="GND"/>
-<wire x1="5.08" y1="58.42" x2="5.08" y2="60.96" width="0.1524" layer="91"/>
-</segment>
 </net>
 <net name="GND_D" class="0">
@@
 <wire x1="-43.18" y1="-40.64" x2="-45.72" y2="-43.18" width="0.1524" layer="91"/>
 </segment>
-</net>
+<segment>
+<pinref part="U1" gate="A" pin="GND"/>
+<pinref part="GND1" gate="1" pin="GND"/>
+<wire x1="5.08" y1="58.42" x2="5.08" y2="60.96" width="0.1524" layer="91"/>
+</segment>
+</net>
+<net name="N$30" class="0">
+<segment>
+<pinref part="JP10" gate="A" pin="1"/>
+<pinref part="JP3" gate="A" pin="1"/>
+<wire x1="-81.28" y1="12.7" x2="-83.82" y2="12.7" width="0.1524" layer="91"/>
+<pinref part="JP2" gate="A" pin="2"/>
+<wire x1="-83.82" y1="33.02" x2="-86.36" y2="33.02" width="0.1524" layer="91"/>
+<wire x1="-83.82" y1="33.02" x2="-83.82" y2="12.7" width="0.1524" layer="91"/>
+<junction x="-83.82" y="33.02"/>
+<wire x1="-78.74" y1="33.02" x2="-83.82" y2="33.02" width="0.1524" layer="91"/>
+<wire x1="-78.74" y1="33.02" x2="-78.74" y2="27.94" width="0.1524" layer="91"/>
+<wire x1="-78.74" y1="27.94" x2="-73.66" y2="27.94" width="0.1524" layer="91"/>
+</segment>
+</net>
