File: Eagle/ISI_experiement.sch (EAGLE design)
At the start: 63 parts, among them IC1 74AC11374D, IC2 74HC04D, IC3 74AC11374D, IC4 74AC11374D, IC5 74266D, IC6 74266D, IC7 74HC04D

Commit message: really close to final ISI
missing inductor package dimensions and one cap value.
Connections:
- net JNC renamed VCC_3V
- removed net VCC-5V: IC6P.VCC
- removed net VCC_5V: C2.1, C3.1, C4.1, C5.1, C6.1, IC1P.VCC@2, IC2P.VCC, IC3P.VCC@2, IC4P.VCC@2, IC5P.VCC, IC7P.VCC, R1.1, SJ1.2, U$1.IN, USBMINI.VBUS
- net GND: now also C2.2, DELP.GND@4, IC1A.OC, IC3A.OC, IC4A.OC
- net VCC: now also C2.1, C3.1, C4.1, C5.1, C6.1, DELP.VCC@2, IC1P.VCC@2, IC2P.VCC, IC3P.VCC@2, IC4P.VCC@2, IC5P.VCC, IC6P.VCC, IC7P.VCC, R1.1, SJ1.2, U$1.IN, USBMINI.VBUS
Changed lines of the file:
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@@
 <instance part="SJ1" gate="1" x="215.9" y="185.42" rot="R90"/>
 <instance part="SJ2" gate="1" x="388.62" y="195.58" rot="R90"/>
-<instance part="GND14" gate="1" x="193.04" y="185.42"/>
+<instance part="GND14" gate="1" x="193.04" y="182.88"/>
 <instance part="GND13" gate="1" x="205.74" y="182.88"/>
 <instance part="IC7" gate="A" x="33.02" y="33.02"/>
@@
 <instance part="RC8" gate="G$1" x="368.3" y="109.22" rot="R180"/>
 <instance part="RC9" gate="G$1" x="368.3" y="101.6" rot="R180"/>
+<instance part="DEL" gate="P" x="365.76" y="83.82"/>
+<instance part="COUNTER" gate="P" x="350.52" y="83.82"/>
 </instances>
 <busses>
@@
 <pinref part="IC1" gate="A" pin="Q2"/>
 <wire x1="48.26" y1="248.92" x2="43.18" y2="248.92" width="0.1524" layer="91"/>
+<label x="43.18" y="248.92" size="1.778" layer="95"/>
 </segment>
 </net>
@@
 <pinref part="JP8" gate="A" pin="1"/>
 <wire x1="17.78" y1="129.54" x2="12.7" y2="129.54" width="0.1524" layer="91"/>
+<label x="7.62" y="129.54" size="1.778" layer="95"/>
 </segment>
 </net>
@@
 <segment>
 <pinref part="IC7" gate="P" pin="GND"/>
-<wire x1="15.24" y1="43.18" x2="22.86" y2="45.72" width="0.1524" layer="91"/>
+<wire x1="15.24" y1="43.18" x2="17.78" y2="43.18" width="0.1524" layer="91"/>
+<label x="17.78" y="40.64" size="1.778" layer="95"/>
 </segment>
 <segment>
@@
 <pinref part="GND22" gate="1" pin="GND"/>
 </segment>
-</net>
-<net name="JNC" class="0">
+<segment>
+<pinref part="DEL" gate="P" pin="GND@4"/>
+<wire x1="373.38" y1="76.2" x2="373.38" y2="73.66" width="0.1524" layer="91"/>
+<label x="373.38" y="73.66" size="1.778" layer="95"/>
+</segment>
+<segment>
+<pinref part="C2" gate="G$1" pin="2"/>
+<pinref part="GND14" gate="1" pin="GND"/>
+</segment>
+<segment>
+<pinref part="IC1" gate="A" pin="OC"/>
+<wire x1="17.78" y1="228.6" x2="12.7" y2="228.6" width="0.1524" layer="91"/>
+<label x="12.7" y="228.6" size="1.778" layer="95"/>
+</segment>
+<segment>
+<pinref part="IC3" gate="A" pin="OC"/>
+<wire x1="17.78" y1="193.04" x2="12.7" y2="193.04" width="0.1524" layer="91"/>
+<label x="12.7" y="193.04" size="1.778" layer="95"/>
+</segment>
+<segment>
+<pinref part="IC4" gate="A" pin="OC"/>
+<wire x1="17.78" y1="157.48" x2="15.24" y2="157.48" width="0.1524" layer="91"/>
+<label x="12.7" y="157.48" size="1.778" layer="95"/>
+</segment>
+</net>
+<net name="VCC_3V" class="0">
 <segment>
 <pinref part="U$1" gate="G$1" pin="OUT"/>
@@
 </segment>
 </net>
-<net name="VCC_5V" class="0">
+<net name="N$5" class="0">
+<segment>
+<pinref part="U$2" gate="G$1" pin="TRI-STATE"/>
+<wire x1="210.82" y1="81.28" x2="210.82" y2="73.66" width="0.1524" layer="91"/>
+<wire x1="210.82" y1="73.66" x2="185.42" y2="73.66" width="0.1524" layer="91"/>
+<pinref part="RC1" gate="G$1" pin="1"/>
+<wire x1="185.42" y1="73.66" x2="185.42" y2="93.98" width="0.1524" layer="91"/>
+</segment>
+</net>
+<net name="VCC" class="0">
+<segment>
+<pinref part="RC1" gate="G$1" pin="2"/>
+<wire x1="185.42" y1="104.14" x2="185.42" y2="129.54" width="0.1524" layer="91"/>
+<wire x1="185.42" y1="129.54" x2="226.06" y2="129.54" width="0.1524" layer="91"/>
+<wire x1="226.06" y1="129.54" x2="226.06" y2="121.92" width="0.1524" layer="91"/>
+<wire x1="226.06" y1="121.92" x2="226.06" y2="119.38" width="0.1524" layer="91"/>
+<wire x1="226.06" y1="129.54" x2="226.06" y2="134.62" width="0.1524" layer="91"/>
+<pinref part="P+1" gate="VCC" pin="VCC"/>
+<junction x="226.06" y="129.54"/>
+<pinref part="U$2" gate="G$1" pin="VCC"/>
+<junction x="226.06" y="121.92"/>
+</segment>
+<segment>
+<pinref part="COUNTER" gate="A" pin="LD"/>
+<wire x1="254" y1="91.44" x2="241.3" y2="91.44" width="0.1524" layer="91"/>
+<wire x1="241.3" y1="91.44" x2="241.3" y2="134.62" width="0.1524" layer="91"/>
+<pinref part="P+2" gate="VCC" pin="VCC"/>
+</segment>
 <segment>
 <pinref part="USBMINI" gate="G$1" pin="VBUS"/>
@@
 <junction x="193.04" y="195.58"/>
 <junction x="261.62" y="195.58"/>
+<label x="185.42" y="198.12" size="1.778" layer="95"/>
+</segment>
+<segment>
+<pinref part="IC1" gate="P" pin="VCC@2"/>
+<wire x1="91.44" y1="261.62" x2="91.44" y2="264.16" width="0.1524" layer="91"/>
+<label x="91.44" y="264.16" size="1.778" layer="95"/>
+</segment>
+<segment>
+<pinref part="IC3" gate="P" pin="VCC@2"/>
+<wire x1="106.68" y1="261.62" x2="106.68" y2="264.16" width="0.1524" layer="91"/>
+<label x="106.68" y="264.16" size="1.778" layer="95"/>
+</segment>
+<segment>
+<pinref part="IC4" gate="P" pin="VCC@2"/>
+<wire x1="121.92" y1="261.62" x2="121.92" y2="264.16" width="0.1524" layer="91"/>
+<label x="121.92" y="264.16" size="1.778" layer="95"/>
+</segment>
+<segment>
+<pinref part="IC5" gate="P" pin="VCC"/>
+<wire x1="93.98" y1="231.14" x2="93.98" y2="233.68" width="0.1524" layer="91"/>
+<label x="93.98" y="233.68" size="1.778" layer="95"/>
+</segment>
+<segment>
+<pinref part="IC6" gate="P" pin="VCC"/>
+<wire x1="111.76" y1="180.34" x2="111.76" y2="185.42" width="0.1524" layer="91"/>
+<label x="111.76" y="185.42" size="1.778" layer="95"/>
 </segment>
 <segment>
@@
 <segment>
 <pinref part="IC7" gate="P" pin="VCC"/>
-<wire x1="15.24" y1="58.42" x2="22.86" y2="58.42" width="0.1524" layer="91"/>
+<wire x1="15.24" y1="58.42" x2="17.78" y2="58.42" width="0.1524" layer="91"/>
 <label x="20.32" y="55.88" size="1.778" layer="95"/>
 </segment>
 <segment>
-<pinref part="IC5" gate="P" pin="VCC"/>
-<wire x1="93.98" y1="231.14" x2="93.98" y2="233.68" width="0.1524" layer="91"/>
-<label x="93.98" y="233.68" size="1.778" layer="95"/>
-</segment>
-<segment>
-<pinref part="IC1" gate="P" pin="VCC@2"/>
-<wire x1="91.44" y1="261.62" x2="91.44" y2="264.16" width="0.1524" layer="91"/>
-<label x="91.44" y="264.16" size="1.778" layer="95"/>
-</segment>
-<segment>
-<pinref part="IC3" gate="P" pin="VCC@2"/>
-<wire x1="106.68" y1="261.62" x2="106.68" y2="264.16" width="0.1524" layer="91"/>
-<label x="106.68" y="264.16" size="1.778" layer="95"/>
-</segment>
-<segment>
-<pinref part="IC4" gate="P" pin="VCC@2"/>
-<wire x1="121.92" y1="261.62" x2="121.92" y2="264.16" width="0.1524" layer="91"/>
-<label x="121.92" y="264.16" size="1.778" layer="95"/>
-</segment>
-</net>
-<net name="VCC-5V" class="0">
-<segment>
-<pinref part="IC6" gate="P" pin="VCC"/>
-<wire x1="111.76" y1="180.34" x2="111.76" y2="185.42" width="0.1524" layer="91"/>
-<label x="111.76" y="185.42" size="1.778" layer="95"/>
-</segment>
-</net>
-<net name="N$5" class="0">
-<segment>
-<pinref part="U$2" gate="G$1" pin="TRI-STATE"/>
-<wire x1="210.82" y1="81.28" x2="210.82" y2="73.66" width="0.1524" layer="91"/>
-<wire x1="210.82" y1="73.66" x2="185.42" y2="73.66" width="0.1524" layer="91"/>
-<pinref part="RC1" gate="G$1" pin="1"/>
-<wire x1="185.42" y1="73.66" x2="185.42" y2="93.98" width="0.1524" layer="91"/>
-</segment>
-</net>
-<net name="VCC" class="0">
-<segment>
-<pinref part="RC1" gate="G$1" pin="2"/>
-<wire x1="185.42" y1="104.14" x2="185.42" y2="129.54" width="0.1524" layer="91"/>
-<wire x1="185.42" y1="129.54" x2="226.06" y2="129.54" width="0.1524" layer="91"/>
-<wire x1="226.06" y1="129.54" x2="226.06" y2="121.92" width="0.1524" layer="91"/>
-<wire x1="226.06" y1="121.92" x2="226.06" y2="119.38" width="0.1524" layer="91"/>
-<wire x1="226.06" y1="129.54" x2="226.06" y2="134.62" width="0.1524" layer="91"/>
-<pinref part="P+1" gate="VCC" pin="VCC"/>
-<junction x="226.06" y="129.54"/>
-<pinref part="U$2" gate="G$1" pin="VCC"/>
-<junction x="226.06" y="121.92"/>
-</segment>
-<segment>
-<pinref part="COUNTER" gate="A" pin="LD"/>
-<wire x1="254" y1="91.44" x2="241.3" y2="91.44" width="0.1524" layer="91"/>
-<wire x1="241.3" y1="91.44" x2="241.3" y2="134.62" width="0.1524" layer="91"/>
-<pinref part="P+2" gate="VCC" pin="VCC"/>
+<pinref part="DEL" gate="P" pin="VCC@2"/>
+<wire x1="368.3" y1="91.44" x2="368.3" y2="93.98" width="0.1524" layer="91"/>
+<label x="368.3" y="91.44" size="1.778" layer="95"/>
 </segment>
 </net>
@@
 <junction x="327.66" y="109.22"/>
 <junction x="327.66" y="111.76"/>
+<junction x="327.66" y="114.3"/>
 </segment>
 </net>
@@
 </sheet>
 </sheets>
+<errors>
+</errors>
 </schematic>
 </drawing>

Commit message: Updated ISI schematic and board
Parts:
- removed C1: (no value), c-trimm:C-TRIMM3008
- removed JP1, JP2, JP3: (no value), jumper:JP1E
- removed L1: SMF51-2-51-15, inductor-neosid:SMF51-2-51-15
- removed SJ1, SJ2: (no value), jumper:SJW
- removed TP$1, TP$10, TP$3, TP$4, TP$5, TP$6, TP$7, TP$8, TP$9: JP1, E3VB_ISI:JP1
- added JP10, JP7, JPC, JPL, JPR: (no value), jumper:JP1E
- renumbered C2 to CP1, C3 to CP2, C4 to CP3, C5 to CP4, C6 to CP5, C7 to CP6, C8 to CP8, C9 to CP7, JP11 to INA2, JP4 to INV, JP5 to INA4, JP8 to INA1, JP9 to INA3, R1 to RP1, R2 to RP2, R3 to RP3, R4 to RP4, TP$2 to V, TP1 to OUTA1, TP2 to OUTA2, TP3 to OUTV, TP4 to OUTA3, TP5 to OUTA4
Connections:
- net N$24 renamed OUTA4
- removed net N$18: C1.A, JP2.2
- net GND: now also JP10.1, JP7.1, JPC.1; no longer JP2.1, SJ1.1, SJ2.1
- net N$1: now also IC7A.O, JPR.1; no longer JP3.2, L1G$1.A
- net N$11: no longer TP$5.1, TP$6.1
- net N$16: no longer TP$7.1, TP$8.1
- net N$3: now also JPL.1, JPR.2; no longer C1.E, IC7A.O, JP1.1, L1G$1.E, TP$1.1
- net N$4: now also JPC.2, JPL.2; no longer JP1.2, JP3.1
- net N$7: no longer TP$3.1, TP$4.1
- net N$8: no longer TP$10.1, TP$9.1
- net VCC: now also JP7.2; no longer SJ1.2
- net VCC_3V: now also JP10.2; no longer SJ2.2
Other:
- note added: "C"
- note added: "L"
- note added: "R"

Commit message: ISI updated
Still need to make 2 parts but that should no affect routing of LFSR.
Parts:
- removed JPR: (no value), jumper:JP1E
- added JPL1, JPL2, JPL3: (no value), jumper:JP1E
- added L1, L3: (no value), rcl:L-USL1812
- added L2: SMF51-2-51-51, inductor-neosid:SMF51-2-51-51
- added TPA1S, TPA2S, TPA3S, TPA4S, TPA4S1, TPA4S2, TPA4S3, TPA4S4: JP1, E3VB_ISI:JP1
- renumbered DEL to BUFFER, RC9 to NP
Connections:
- net N$6 renamed CRY_OUT
- new net N$18: JPL2.2, L1.1
- new net N$24: JPL1.2, L3.1
- net N$1: now also JPL.1, JPL1.1, JPL2.1, JPL3.1; no longer JPR.1
- net N$11: now also TPA2S.1, TPA4S3.1
- net N$16: now also TPA3S.1, TPA4S2.1
- net N$3: now also JPL3.2, L2G$1.A; no longer JPL.1, JPR.2
- net N$4: now also L1.2, L2G$1.E, L3.2
- net N$7: now also TPA1S.1, TPA4S4.1
- net N$8: now also TPA4S.1, TPA4S1.1
Other:
- note removed: "R"
- moved on the sheet: C_GND

Commit message: first run full layout of isi board
Parts:
- removed CP6: 18pF, adafruit:C-USC1206K
- removed CP7: 100uF, adafruit:C-USC1206K
- removed CP8: 10uF, adafruit:C-USC1206K
- removed C_GND, TPA1S, TPA2S, TPA3S, TPA4S, TPA4S1, TPA4S2, TPA4S3, TPA4S4, V: JP1, E3VB_ISI:JP1
- removed JP10: (no value), jumper:JP1E
- removed LED1: (no value), adafruit:LEDCHIPLED_0805
- removed RP1: 1K, adafruit:R-US_R0805
- removed RP2: 51K, adafruit:R-US_R0805
- removed RP3: 30K, adafruit:R-US_R0805
- removed RP4: 220, adafruit:R-US_R0805
- removed U$1: TPS796, Capstone:TPS796
- added U$3: C-TRIMM, E3VB_ISI:C-TRIMM
- CP1, CP3, CP4: value 100uF -> (none)
- CP2: value 10uF -> (none)
- CP5: value 0.1uF -> (none)
Connections:
- removed net N$1: IC7A.O, JPL.1, JPL1.1, JPL2.1, JPL3.1
- removed net N$10: RP1.2, U$1.EN
- removed net N$11: IC2C.O, IC2D.I, TPA2S.1, TPA4S3.1
- removed net N$12: CP6.2, RP2.1, RP3.2, U$1.NR/FB
- removed net N$13: LED1.C, RP4.2
- removed net N$16: IC2E.O, IC2F.I, TPA3S.1, TPA4S2.1
- removed net N$7: IC2A.O, IC2B.I, TPA1S.1, TPA4S4.1
- removed net N$8: IC7C.O, IC7D.I, TPA4S.1, TPA4S1.1
- removed net VCC_3V: CP6.1, CP7.1, CP8.1, JP10.2, LED1.A, RP2.2, U$1.OUT
- new net 1: IC2C.O, IC7B.I
- new net 2: IC2B.O, IC7A.I
- new net 3: IC2D.O, IC7D.I
- new net 4: IC2E.O, IC7E.I
- new net V: IC2A.O, JPL.1, JPL1.1, JPL2.1, JPL3.1
- net CLK2: now also IC4A.CLK; no longer IC3A.CLK
- net CLK3: now also IC3A.CLK; no longer IC4A.CLK
- net GND: now also U$3.G, U$3.P; no longer CP7.2, CP8.2, C_GND.1, JP10.1, RP3.1, RP4.1, U$1.6, U$1.GND
- net N$14: now also IC2C.I; no longer IC2A.I
- net N$17: now also IC7C.O; no longer IC7B.O
- net N$19: now also IC7E.O; no longer IC7D.O
- net N$2: now also IC2B.I, INA2.2; no longer IC7A.I, INV.2
- net N$20: now also IC7A.O; no longer IC2D.O
- net N$21: now also IC2E.I; no longer IC7C.I
- net N$22: now also IC2A.I, INV.2; no longer IC2C.I, INA2.2
- net N$25: now also IC2D.I; no longer IC2E.I
- net N$28: now also JP6.5; no longer JP6.1
- net N$29: now also JP6.3; no longer JP6.5
- net N$30: now also JP6.7; no longer JP6.3
- net N$31: now also JP6.1; no longer JP6.7
- net N$4: now also IC7C.I; no longer IC7B.I, V.1
- net N$9: now also IC7B.O; no longer IC2B.O
- net OUTA4: now also IC7D.O; no longer IC2F.O
- net VCC: no longer RP1.1, U$1.IN
Other:
- note removed: "3.3V Test Point"
- moved on the sheet: IC2A, IC2B, IC2C, IC2D, IC2E, IC7A, IC7B, IC7C, IC7D, JPC, L2

Commit message: upload latest isi board
Parts:
- renumbered U$2 to U$1
Changed lines of the file:
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@@
 <part name="GND20" library="supply1" deviceset="GND" device=""/>
 <part name="GND21" library="supply1" deviceset="GND" device=""/>
-<part name="U$2" library="Capstone" deviceset="ECS-8FX" device=""/>
 <part name="COUNTER" library="74xx-eu" deviceset="74*191" device="N" technology="HC"/>
 <part name="BUFFER" library="74ac-logic" deviceset="74AC11240" device="D"/>
@@
 <part name="U$3" library="E3VB_ISI" deviceset="C-TRIMM" device=""/>
 <part name="GND25" library="supply1" deviceset="GND" device=""/>
+<part name="U$1" library="Capstone" deviceset="ECS-8FX" device=""/>
 </parts>
 <sheets>
@@
 <instance part="GND20" gate="1" x="111.76" y="241.3"/>
 <instance part="GND21" gate="1" x="127" y="241.3"/>
-<instance part="U$2" gate="G$1" x="231.14" y="119.38" rot="R90"/>
 <instance part="COUNTER" gate="A" x="266.7" y="101.6"/>
 <instance part="BUFFER" gate="A" x="342.9" y="109.22"/>
@@
 <instance part="U$3" gate="G$1" x="104.14" y="20.32"/>
 <instance part="GND25" gate="1" x="104.14" y="12.7"/>
+<instance part="U$1" gate="G$1" x="231.14" y="119.38" rot="R90"/>
 </instances>
 <busses>
@@
 </segment>
 <segment>
-<pinref part="U$2" gate="G$1" pin="GND"/>
 <wire x1="226.06" y1="81.28" x2="226.06" y2="76.2" width="0.1524" layer="91"/>
 <pinref part="GND22" gate="1" pin="GND"/>
+<pinref part="U$1" gate="G$1" pin="GND"/>
 </segment>
 <segment>
@@
 <net name="N$5" class="0">
 <segment>
-<pinref part="U$2" gate="G$1" pin="TRI-STATE"/>
 <wire x1="210.82" y1="81.28" x2="210.82" y2="73.66" width="0.1524" layer="91"/>
 <wire x1="210.82" y1="73.66" x2="185.42" y2="73.66" width="0.1524" layer="91"/>
 <pinref part="RC1" gate="G$1" pin="1"/>
 <wire x1="185.42" y1="73.66" x2="185.42" y2="93.98" width="0.1524" layer="91"/>
+<pinref part="U$1" gate="G$1" pin="TRI-STATE"/>
 </segment>
 </net>
@@
 <pinref part="P+1" gate="VCC" pin="VCC"/>
 <junction x="226.06" y="129.54"/>
-<pinref part="U$2" gate="G$1" pin="VCC"/>
+<pinref part="U$1" gate="G$1" pin="VCC"/>
 <junction x="226.06" y="121.92"/>
 </segment>
@@
 <net name="CRY_OUT" class="0">
 <segment>
-<pinref part="U$2" gate="G$1" pin="OUTPUT"/>
 <wire x1="210.82" y1="121.92" x2="210.82" y2="124.46" width="0.1524" layer="91"/>
 <wire x1="210.82" y1="124.46" x2="238.76" y2="124.46" width="0.1524" layer="91"/>
@@
 <pinref part="COUNTER" gate="A" pin="CLK"/>
 <wire x1="238.76" y1="99.06" x2="254" y2="99.06" width="0.1524" layer="91"/>
-</segment>
-</net>
+<pinref part="U$1" gate="G$1" pin="OUTPUT"/>
+</segment>
+</net>

Commit message: some changes to the traces
Parts:
- L2: value SMF51-2-51-51 -> RF_INDUCTOR; device inductor-neosid:SMF51-2-51-51 -> E3VB_ISI:RF_INDUCTOR
- renumbered IC2 to VCC
Connections:
- net V renamed V1
- new net N$8: JPC.1, U$3.P
- net 1: now also IC7E.I, VCCE.O; no longer IC7B.I, VCCC.O
- net 4: now also IC7B.I, VCCC.O; no longer IC7E.I, VCCE.O
- net GND: no longer JPC.1, U$3.P
- net N$3: now also L2.A1; no longer L2G$1.A
- net N$4: now also L2.E1; no longer L2G$1.E
Other:
- moved on the sheet: L2
Changed lines of the file:
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@@
 <?xml version="1.0" encoding="utf-8"?>
 <!DOCTYPE eagle SYSTEM "eagle.dtd">
-<eagle version="7.1.0">
+<eagle version="7.2.0">
 <drawing>
 <settings>
@@
 <part name="INV" library="jumper" deviceset="JP1E" device=""/>
 <part name="OUTA1" library="E3VB_ISI" deviceset="JP1" device=""/>
-<part name="IC2" library="74xx-eu" deviceset="74*04" device="D" technology="HC"/>
+<part name="VCC" library="74xx-eu" deviceset="74*04" device="D" technology="HC"/>
 <part name="INA1" library="jumper" deviceset="JP1E" device=""/>
 <part name="OUTA2" library="E3VB_ISI" deviceset="JP1" device=""/>
@@
 <part name="L1" library="rcl" deviceset="L-US" device="L1812"/>
 <part name="L3" library="rcl" deviceset="L-US" device="L1812"/>
-<part name="L2" library="inductor-neosid" deviceset="SMF51-2-" device="51-51"/>
+<part name="L2" library="E3VB_ISI" deviceset="RF_INDUCTOR" device=""/>
 <part name="U$3" library="E3VB_ISI" deviceset="C-TRIMM" device=""/>
 <part name="GND25" library="supply1" deviceset="GND" device=""/>
@@
 <instance part="IC7" gate="P" x="15.24" y="50.8"/>
 <instance part="OUTA1" gate="G$1" x="144.78" y="134.62"/>
-<instance part="IC2" gate="A" x="33.02" y="33.02"/>
+<instance part="VCC" gate="A" x="33.02" y="33.02"/>
 <instance part="INA1" gate="A" x="17.78" y="132.08"/>
 <instance part="OUTA2" gate="G$1" x="144.78" y="114.3"/>
@@
 <instance part="OUTA4" gate="G$1" x="144.78" y="78.74"/>
 <instance part="INA4" gate="A" x="17.78" y="76.2"/>
-<instance part="IC2" gate="P" x="162.56" y="127"/>
+<instance part="VCC" gate="P" x="162.56" y="127"/>
 <instance part="IC6" gate="P" x="111.76" y="170.18"/>
 <instance part="IC5" gate="P" x="93.98" y="220.98"/>
@@
 <instance part="L1" gate="G$1" x="91.44" y="48.26" rot="R90"/>
 <instance part="L3" gate="G$1" x="91.44" y="40.64" rot="R90"/>
-<instance part="L2" gate="G$1" x="91.44" y="60.96" rot="R90"/>
-<instance part="IC2" gate="B" x="38.1" y="109.22"/>
-<instance part="IC2" gate="C" x="38.1" y="129.54"/>
-<instance part="IC2" gate="D" x="38.1" y="88.9"/>
-<instance part="IC2" gate="E" x="38.1" y="73.66"/>
+<instance part="L2" gate="G$1" x="91.44" y="58.42" rot="R90"/>
+<instance part="VCC" gate="B" x="38.1" y="109.22"/>
+<instance part="VCC" gate="C" x="38.1" y="129.54"/>
+<instance part="VCC" gate="D" x="38.1" y="88.9"/>
+<instance part="VCC" gate="E" x="38.1" y="73.66"/>
 <instance part="IC7" gate="B" x="127" y="129.54"/>
 <instance part="IC7" gate="C" x="121.92" y="33.02"/>
@@
 </segment>
 <segment>
-<pinref part="JPC" gate="A" pin="1"/>
-<wire x1="104.14" y1="25.4" x2="104.14" y2="22.86" width="0.1524" layer="91"/>
-<pinref part="U$3" gate="G$1" pin="P"/>
-</segment>
-<segment>
-<pinref part="IC2" gate="P" pin="GND"/>
+<pinref part="VCC" gate="P" pin="GND"/>
 <wire x1="162.56" y1="119.38" x2="162.56" y2="116.84" width="0.1524" layer="91"/>
 <pinref part="GND15" gate="1" pin="GND"/>
@@
 <wire x1="99.06" y1="33.02" x2="104.14" y2="33.02" width="0.1524" layer="91"/>
 <pinref part="JPL" gate="A" pin="2"/>
-<pinref part="L2" gate="G$1" pin="E"/>
-<wire x1="93.98" y1="58.42" x2="99.06" y2="55.88" width="0.1524" layer="91"/>
+<pinref part="L2" gate="G$1" pin="E1"/>
+<wire x1="93.98" y1="55.88" x2="99.06" y2="55.88" width="0.1524" layer="91"/>
 <wire x1="99.06" y1="55.88" x2="99.06" y2="48.26" width="0.1524" layer="91"/>
 <junction x="99.06" y="33.02"/>
@@
 </segment>
 </net>
-<net name="1" class="0">
+<net name="4" class="0">
 <segment>
 <wire x1="48.26" y1="129.54" x2="116.84" y2="129.54" width="0.1524" layer="91"/>
 <pinref part="IC7" gate="B" pin="I"/>
-<pinref part="IC2" gate="C" pin="O"/>
+<pinref part="VCC" gate="C" pin="O"/>
 </segment>
 </net>
@@
 <wire x1="48.26" y1="109.22" x2="116.84" y2="109.22" width="0.1524" layer="91"/>
 <pinref part="IC7" gate="A" pin="I"/>
-<pinref part="IC2" gate="B" pin="O"/>
+<pinref part="VCC" gate="B" pin="O"/>
 </segment>
 </net>
@@
 <segment>
 <wire x1="48.26" y1="88.9" x2="116.84" y2="88.9" width="0.1524" layer="91"/>
-<pinref part="IC2" gate="D" pin="O"/>
+<pinref part="VCC" gate="D" pin="O"/>
 <pinref part="IC7" gate="D" pin="I"/>
 </segment>
@@
 <pinref part="INA3" gate="A" pin="2"/>
 <wire x1="20.32" y1="88.9" x2="27.94" y2="88.9" width="0.1524" layer="91"/>
-<pinref part="IC2" gate="D" pin="I"/>
-</segment>
-</net>
-<net name="4" class="0">
+<pinref part="VCC" gate="D" pin="I"/>
+</segment>
+</net>
+<net name="1" class="0">
 <segment>
 <wire x1="48.26" y1="73.66" x2="116.84" y2="73.66" width="0.1524" layer="91"/>
-<pinref part="IC2" gate="E" pin="O"/>
+<pinref part="VCC" gate="E" pin="O"/>
 <pinref part="IC7" gate="E" pin="I"/>
 </segment>
@@
 <pinref part="INA4" gate="A" pin="2"/>
 <wire x1="20.32" y1="73.66" x2="27.94" y2="73.66" width="0.1524" layer="91"/>
-<pinref part="IC2" gate="E" pin="I"/>
+<pinref part="VCC" gate="E" pin="I"/>
 </segment>
 </net>
@@
 </segment>
 <segment>
-<pinref part="IC2" gate="P" pin="VCC"/>
+<pinref part="VCC" gate="P" pin="VCC"/>
 <wire x1="162.56" y1="134.62" x2="162.56" y2="137.16" width="0.1524" layer="91"/>
 <label x="162.56" y="137.16" size="1.778" layer="95"/>
@@
 </segment>
 </net>
-<net name="N$27" class="0">
+<net name="N$7" class="0">
 <segment>
 <pinref part="COUNTER" gate="A" pin="QD"/>
@@
 </segment>
 </net>
-<net name="V" class="0">
+<net name="V1" class="0">
 <segment>
 <pinref part="JPL" gate="A" pin="1"/>
@@
 <junction x="76.2" y="48.26"/>
 <wire x1="43.18" y1="33.02" x2="76.2" y2="33.02" width="0.1524" layer="91"/>
-<pinref part="IC2" gate="A" pin="O"/>
+<pinref part="VCC" gate="A" pin="O"/>
 </segment>
 </net>
@@
 <net name="N$3" class="0">
 <segment>
-<pinref part="L2" gate="G$1" pin="A"/>
+<pinref part="L2" gate="G$1" pin="A1"/>
 <pinref part="JPL3" gate="A" pin="2"/>
-<wire x1="86.36" y1="58.42" x2="83.82" y2="55.88" width="0.1524" layer="91"/>
+<wire x1="86.36" y1="55.88" x2="83.82" y2="55.88" width="0.1524" layer="91"/>
 </segment>
 </net>
@@
 <pinref part="INV" gate="A" pin="2"/>
 <wire x1="15.24" y1="33.02" x2="22.86" y2="33.02" width="0.1524" layer="91"/>
-<pinref part="IC2" gate="A" pin="I"/>
+<pinref part="VCC" gate="A" pin="I"/>
 </segment>
 </net>
@@
 <pinref part="INA2" gate="A" pin="2"/>
 <wire x1="20.32" y1="109.22" x2="27.94" y2="109.22" width="0.1524" layer="91"/>
-<pinref part="IC2" gate="B" pin="I"/>
+<pinref part="VCC" gate="B" pin="I"/>
 </segment>
 </net>
@@
 <segment>
 <pinref part="INA1" gate="A" pin="2"/>
-<pinref part="IC2" gate="C" pin="I"/>
+<pinref part="VCC" gate="C" pin="I"/>
 <wire x1="20.32" y1="129.54" x2="27.94" y2="129.54" width="0.1524" layer="91"/>
 </segment>
 </net>
+<net name="N$8" class="0">
+<segment>
+<pinref part="U$3" gate="G$1" pin="P"/>
+<pinref part="JPC" gate="A" pin="1"/>
+<wire x1="104.14" y1="22.86" x2="104.14" y2="25.4" width="0.1524" layer="91"/>
+</segment>
+</net>
