File: Eagle/ISI_experiement.sch (EAGLE design)
At the start: 59 parts, among them IC1 74AC11374D, IC3 74AC11374D, IC4 74AC11374D, IC5 74266D, IC6 74266D, IC7 74HC04D

Commit message: version sent to oshpark
Parts:
- added C1, C2, C3, C4, C5, C6, C7: .1uF, T06_LockBox:C
- added R2, R3, R4, R5: 100, T06_LockBox:R-US_M0805
- COUNTER: value 74HC191N -> 74HC191NS; device 74xx-eu:74HC191N -> 74xx-eu:74HC191NS
- CP1, CP3: value (none) -> 100uf
- CP2, CP4: value (none) -> 10uF
- CP5: value (none) -> .1uF
- L1: value (none) -> .5 nH; device rcl:L-USL1812 -> Bourns_By_element14_Batch_1:PM0805-8N2M-RC
- L3: value (none) -> 1nH; device rcl:L-USL1812 -> Bourns_By_element14_Batch_1:PM0805-8N2M-RC
- renumbered VCC to INVBUFF
Connections:
- removed net 4: FEA1.1, IC7B.I, INVBUFFC.O, NEA1.1
- new net 8: FEA4.1, IC7E.I, INVBUFFE.O, NEA4.1
- new net N$16: IC6D.I0, IC6D.I1, R2.2
- new net N$27: IC6B.I0, IC6B.I1, R3.2
- new net N$37: IC6C.I0, IC6C.I1, R4.2
- new net N$41: IC7F.I, R5.2
- net 1: now also FEA1.1, IC7B.I, INVBUFFC.O, NEA1.1; no longer FEA4.1, IC7E.I, INVBUFFE.O, NEA4.1
- net GND: now also C1.2, C2.2, C3.2, C4.2, C5.2, C6.2, C7.2, L2G$2.1, L2G$3.1, R2.1, R3.1, R4.1, R5.1
- net N$3: now also L2G$1.A1; no longer L2.A1
- net N$4: now also L2G$1.E1; no longer L2.E1
- net VCC: now also C1.1, C2.1, C3.1, C4.1, C5.1, C6.1, C7.1

Commit message: changes to git
Parts:
- L1: value .5 nH -> .5 uH
- L3: value 1nH -> 1uH
Changed lines of the file:
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@@
 <part name="JPL2" library="jumper" deviceset="JP1E" device=""/>
 <part name="JPL3" library="jumper" deviceset="JP1E" device=""/>
-<part name="L1" library="Bourns_By_element14_Batch_1" deviceset="PM0805-8N2M-RC" device="" value=".5 nH"/>
-<part name="L3" library="Bourns_By_element14_Batch_1" deviceset="PM0805-8N2M-RC" device="" value="1nH"/>
+<part name="L1" library="Bourns_By_element14_Batch_1" deviceset="PM0805-8N2M-RC" device="" value=".5 uH"/>
+<part name="L3" library="Bourns_By_element14_Batch_1" deviceset="PM0805-8N2M-RC" device="" value="1uH"/>
 <part name="L2" library="E3VB_ISI" deviceset="RF_INDUCTOR" device=""/>
 <part name="U$3" library="E3VB_ISI" deviceset="C-TRIMM" device=""/>

Commit message: updated boards
fixed some of the issued we encountered while making the board
Parts:
- added C10, C11, C12, C8, C9: 50pf, T06_LockBox:C
- added R1, R6, R7, R8, R9: 1K, T06_LockBox:R-US_M0805
Connections:
- net FB0: now also C12.1, R9.1
- net FB1: now also C11.1, R8.1
- net FB2: now also C10.1, R7.1
- net FB3: now also C9.1, R6.1
- net FB4: now also C8.1, R1.1
- net GND: now also C10.2, C11.2, C12.2, C8.2, C9.2
- net VCC: now also R1.2, R6.2, R7.2, R8.2, R9.2
Changed lines of the file:
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@@
 <part name="R5" library="T06_LockBox" deviceset="R-US_" device="M0805" value="100"/>
 <part name="GND12" library="supply1" deviceset="GND" device=""/>
+<part name="R1" library="T06_LockBox" deviceset="R-US_" device="M0805" value="1K"/>
+<part name="R6" library="T06_LockBox" deviceset="R-US_" device="M0805" value="1K"/>
+<part name="R7" library="T06_LockBox" deviceset="R-US_" device="M0805" value="1K"/>
+<part name="R8" library="T06_LockBox" deviceset="R-US_" device="M0805" value="1K"/>
+<part name="R9" library="T06_LockBox" deviceset="R-US_" device="M0805" value="1K"/>
+<part name="C8" library="T06_LockBox" deviceset="C" device="" value="50pf"/>
+<part name="C9" library="T06_LockBox" deviceset="C" device="" value="50pf"/>
+<part name="C10" library="T06_LockBox" deviceset="C" device="" value="50pf"/>
+<part name="C11" library="T06_LockBox" deviceset="C" device="" value="50pf"/>
+<part name="C12" library="T06_LockBox" deviceset="C" device="" value="50pf"/>
 </parts>
 <sheets>
@@
 <instance part="R5" gate="G$1" x="345.44" y="203.2" rot="R90"/>
 <instance part="GND12" gate="1" x="345.44" y="193.04"/>
+<instance part="R1" gate="G$1" x="83.82" y="182.88" rot="R90"/>
+<instance part="R6" gate="G$1" x="83.82" y="203.2" rot="R90"/>
+<instance part="R7" gate="G$1" x="86.36" y="218.44" rot="R90"/>
+<instance part="R8" gate="G$1" x="78.74" y="236.22" rot="R90"/>
+<instance part="R9" gate="G$1" x="78.74" y="256.54" rot="R90"/>
+<instance part="C8" gate="G$1" x="83.82" y="175.26"/>
+<instance part="C9" gate="G$1" x="83.82" y="195.58"/>
+<instance part="C10" gate="G$1" x="86.36" y="210.82"/>
+<instance part="C11" gate="G$1" x="78.74" y="228.6"/>
+<instance part="C12" gate="G$1" x="78.74" y="248.92"/>
 </instances>
 <busses>
@@
 <wire x1="76.2" y1="251.46" x2="78.74" y2="251.46" width="0.1524" layer="91"/>
 <label x="78.74" y="251.46" size="1.778" layer="95"/>
+<pinref part="C12" gate="G$1" pin="1"/>
+<pinref part="R9" gate="G$1" pin="1"/>
+<junction x="78.74" y="251.46"/>
 </segment>
 <segment>
@@
 <wire x1="104.14" y1="210.82" x2="93.98" y2="210.82" width="0.1524" layer="91"/>
 <junction x="93.98" y="210.82"/>
+<pinref part="C10" gate="G$1" pin="2"/>
+<wire x1="86.36" y1="205.74" x2="91.44" y2="205.74" width="0.1524" layer="91"/>
+<wire x1="91.44" y1="205.74" x2="91.44" y2="210.82" width="0.1524" layer="91"/>
+<wire x1="91.44" y1="210.82" x2="93.98" y2="210.82" width="0.1524" layer="91"/>
 </segment>
 <segment>
@@
 <wire x1="345.44" y1="195.58" x2="345.44" y2="198.12" width="0.1524" layer="91"/>
 </segment>
+<segment>
+<pinref part="C8" gate="G$1" pin="2"/>
+<wire x1="83.82" y1="170.18" x2="86.36" y2="170.18" width="0.1524" layer="91"/>
+<label x="86.36" y="170.18" size="1.778" layer="95" rot="R270" xref="yes"/>
+</segment>
+<segment>
+<pinref part="C9" gate="G$1" pin="2"/>
+<wire x1="83.82" y1="190.5" x2="86.36" y2="190.5" width="0.1524" layer="91"/>
+<label x="86.36" y="190.5" size="1.778" layer="95" xref="yes"/>
+</segment>
+<segment>
+<pinref part="C11" gate="G$1" pin="2"/>
+<wire x1="78.74" y1="223.52" x2="81.28" y2="223.52" width="0.1524" layer="91"/>
+<wire x1="78.74" y1="223.52" x2="76.2" y2="223.52" width="0.1524" layer="91"/>
+<junction x="78.74" y="223.52"/>
+<label x="76.2" y="223.52" size="1.778" layer="95" rot="R180" xref="yes"/>
+</segment>
+<segment>
+<pinref part="C12" gate="G$1" pin="2"/>
+<wire x1="78.74" y1="243.84" x2="81.28" y2="243.84" width="0.1524" layer="91"/>
+<label x="81.28" y="243.84" size="1.778" layer="95" rot="R180" xref="yes"/>
+</segment>
 </net>
 <net name="N$4" class="0">
@@
 <segment>
 <pinref part="IC5" gate="B" pin="O"/>
-<wire x1="76.2" y1="236.22" x2="78.74" y2="236.22" width="0.1524" layer="91"/>
+<wire x1="76.2" y1="236.22" x2="78.74" y2="231.14" width="0.1524" layer="91"/>
 <label x="78.74" y="236.22" size="1.778" layer="95"/>
+<pinref part="C11" gate="G$1" pin="1"/>
+<pinref part="R8" gate="G$1" pin="1"/>
+<junction x="78.74" y="231.14"/>
 </segment>
 <segment>
@@
 <wire x1="81.28" y1="213.36" x2="86.36" y2="213.36" width="0.1524" layer="91"/>
 <label x="81.28" y="213.36" size="1.778" layer="95"/>
+<pinref part="C10" gate="G$1" pin="1"/>
+<pinref part="R7" gate="G$1" pin="1"/>
+<junction x="86.36" y="213.36"/>
 </segment>
 <segment>
@@
 <wire x1="78.74" y1="198.12" x2="83.82" y2="198.12" width="0.1524" layer="91"/>
 <label x="81.28" y="198.12" size="1.778" layer="95"/>
+<pinref part="C9" gate="G$1" pin="1"/>
+<pinref part="R6" gate="G$1" pin="1"/>
+<junction x="83.82" y="198.12"/>
 </segment>
 <segment>
@@
 <wire x1="78.74" y1="177.8" x2="83.82" y2="177.8" width="0.1524" layer="91"/>
 <label x="81.28" y="177.8" size="1.778" layer="95"/>
+<pinref part="R1" gate="G$1" pin="1"/>
+<pinref part="C8" gate="G$1" pin="1"/>
+<junction x="83.82" y="177.8"/>
 </segment>
 <segment>
@@
 <label x="368.3" y="91.44" size="1.778" layer="95"/>
 </segment>
-</net>
+<segment>
+<pinref part="R9" gate="G$1" pin="2"/>
+<wire x1="78.74" y1="261.62" x2="76.2" y2="261.62" width="0.1524" layer="91"/>
+<wire x1="76.2" y1="261.62" x2="76.2" y2="264.16" width="0.1524" layer="91"/>
+<label x="76.2" y="264.16" size="1.778" layer="95" rot="R180" xref="yes"/>
+</segment>
+<segment>
+<pinref part="R8" gate="G$1" pin="2"/>
+<wire x1="78.74" y1="241.3" x2="76.2" y2="241.3" width="0.1524" layer="91"/>
+<label x="76.2" y="241.3" size="1.778" layer="95" rot="R180" xref="yes"/>
+</segment>
+<segment>
+<pinref part="R7" gate="G$1" pin="2"/>
+<wire x1="86.36" y1="223.52" x2="88.9" y2="223.52" width="0.1524" layer="91"/>
+<label x="88.9" y="223.52" size="1.778" layer="95" rot="R90" xref="yes"/>
+</segment>
+<segment>
+<pinref part="R6" gate="G$1" pin="2"/>
+<wire x1="83.82" y1="208.28" x2="81.28" y2="208.28" width="0.1524" layer="91"/>
+<label x="81.28" y="208.28" size="1.778" layer="95" rot="R180" xref="yes"/>
+</segment>
+<segment>
+<pinref part="R1" gate="G$1" pin="2"/>
+<wire x1="83.82" y1="187.96" x2="81.28" y2="187.96" width="0.1524" layer="91"/>
+<label x="81.28" y="187.96" size="1.778" layer="95" rot="R180" xref="yes"/>
+</segment>
+</net>

Commit message: draft of pass down ISI
missing summary
Other:
- note added: "Date: 6/04/2015"
- note added: "Rev: 1.2"
- note removed: "Date: 4/04/2015"
- note removed: "Rev: 0.3"
Changed lines of the file:
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@@
 <text x="320.04" y="43.18" size="5.08" layer="95">ISI Experiment</text>
 <text x="342.9" y="27.94" size="5.08" layer="95">T12</text>
-<text x="360.68" y="2.54" size="5.08" layer="95">Rev: 0.3</text>
-<text x="309.88" y="2.54" size="3.81" layer="95">Date: 4/04/2015</text>
+<text x="360.68" y="2.54" size="5.08" layer="95">Rev: 1.2</text>
+<text x="309.88" y="2.54" size="3.81" layer="95">Date: 6/04/2015</text>
 <text x="309.88" y="15.24" size="3.81" layer="95">Project: Intel E3V Board/ Capstone Project</text>
 <text x="281.94" y="213.36" size="1.778" layer="91">TPS796 5V to 3.3V Regulator</text>
