File: Eagle/ISIV2/ISI_experiement.brd (EAGLE design)
At the start: 101.6 x 81.3 mm, 59 parts, among them IC1 74AC11374D, IC3 74AC11374D, IC4 74AC11374D, IC5 74266D, IC6 74266D, IC7 74HC04D

Commit message: test board
debug board
Routing:
- net 3: track 456.7 -> 754.0 mm
- net 1: track 439.4 -> 735.6 mm
- net V1: track 427.8 -> 722.6 mm
- net 2: track 408.8 -> 702.2 mm
- net 4: track 406.7 -> 698.7 mm
- net 7: track 23.9 -> 0.00 mm
- net 5: track 23.6 -> 0.00 mm
- net 6: track 21.1 -> 0.00 mm
- net V2: track 19.3 -> 0.00 mm
- net 8: track 12.5 -> 0.00 mm
- net GND: vias 38 -> 44

Commit message: version sent to oshpark
Parts:
- added C1, C2, C3, C4, C5, C6, C7: .1uF, T06_LockBox:C0805
- added R2, R3, R4, R5: 100, T06_LockBox:M0805
- CP1, CP3: value (none) -> 100uf
- CP2, CP4: value (none) -> 10uF
- CP5: value (none) -> .1uF
- L1: value (none) -> .5uH
- L3: value (none) -> 1uH
- moved L2 0.41 mm to (37.3, 25.4), turned to 180 degrees
- moved IC3 0.30 mm to (90.2, 47.2)
Connections:
- removed net 4: FEA1.1, IC7.3, NEA1.1, VCC.6
- new net 8: FEA4.1, IC7.11, NEA4.1, VCC.10
- new net N$16: IC6.12, IC6.13, R2.2
- new net N$27: IC6.5, IC6.6, R3.2
- new net N$37: IC6.8, IC6.9, R4.2
- new net N$41: IC7.13, R5.2
- net 1: now also FEA1.1, IC7.3, NEA1.1, VCC.6; no longer FEA4.1, IC7.11, NEA4.1, VCC.10
- net GND: now also C1.2, C2.2, C3.2, C4.2, C5.2, C6.2, C7.2, L2.P$1, L2.P$5, R2.1, R3.1, R4.1, R5.1
- net N$3: now also L2.P$4; no longer L2.P$2
- net N$4: now also L2.P$2; no longer L2.P$7
- net VCC: now also C1.1, C2.1, C3.1, C4.1, C5.1, C6.1, C7.1
Routing:
- net 4: track 698.7 -> 0.00 mm
- net 8: track 0.00 -> 597.7 mm, vias 0 -> 2
- net 1: track 735.6 -> 560.7 mm, vias 2 -> 0
- net 3: track 754.0 -> 616.0 mm
- net 2: track 702.2 -> 564.2 mm
- net V1: track 722.6 -> 584.7 mm
- net GND: track 66.3 -> 94.2 mm, vias 44 -> 39
- net N$3: track 11.2 -> 4.30 mm
- net N$37: track 0.00 -> 4.88 mm
- net VCC: track 258.2 -> 253.4 mm
- net N$27: track 0.00 -> 4.64 mm
- net N$16: track 0.00 -> 3.42 mm
- net N$41: track 0.00 -> 2.42 mm
