File: Eagle/ISIV2/ISI_experiement.sch (EAGLE design)
At the start: 59 parts, among them IC1 74AC11374D, IC3 74AC11374D, IC4 74AC11374D, IC5 74266D, IC6 74266D, IC7 74HC04D

Commit message: version sent to oshpark
Parts:
- added C1, C2, C3, C4, C5, C6, C7: .1uF, T06_LockBox:C
- added R2, R3, R4, R5: 100, T06_LockBox:R-US_M0805
- CP1, CP3: value (none) -> 100uf
- CP2, CP4: value (none) -> 10uF
- CP5: value (none) -> .1uF
- L1: value (none) -> .5uH
- L3: value (none) -> 1uH
Connections:
- removed net 4: FEA1.1, IC7B.I, NEA1.1, VCCC.O
- new net 8: FEA4.1, IC7E.I, NEA4.1, VCCE.O
- new net N$16: IC6D.I0, IC6D.I1, R2.2
- new net N$27: IC6B.I0, IC6B.I1, R3.2
- new net N$37: IC6C.I0, IC6C.I1, R4.2
- new net N$41: IC7F.I, R5.2
- net 1: now also FEA1.1, IC7B.I, NEA1.1, VCCC.O; no longer FEA4.1, IC7E.I, NEA4.1, VCCE.O
- net GND: now also C1.2, C2.2, C3.2, C4.2, C5.2, C6.2, C7.2, L2G$2.1, L2G$3.1, R2.1, R3.1, R4.1, R5.1
- net N$3: now also L2G$1.A1; no longer L2.A1
- net N$4: now also L2G$1.E1; no longer L2.E1
- net VCC: now also C1.1, C2.1, C3.1, C4.1, C5.1, C6.1, C7.1
Other:
- moved on the sheet: L2G$1
